File: HW/rbpi-z-hat/rbpi-z-hat.sch (KiCad schematic (older format))
At the start: 5 parts, among them Q1 DMG2302U

Commit message: Commit...
Connections:
- net labels added: GNDD
- wire segments 8 -> 12
Changed lines of the file:
@@
 $Descr A4 8268 11693 portrait
 encoding utf-8
-Sheet 1 14
+Sheet 1 18
 Title "RasPi Zero NAV Hat"
 Date "2020-06-08"
@@
 $EndDescr
 $Sheet
-S 5200 2950 650  600
-U 5ED65008
-F0 "MPU9250" 50
-F1 "IMU.sch" 50
-F2 "MPU_MOSI" I L 5200 3050 50
-F3 "MPU_MISO" O L 5200 3150 50
-F4 "MPU_SCLK" I L 5200 3250 50
-F5 "MPU_nCS" I L 5200 3350 50
-F6 "MPU_INT" O L 5200 3450 50
-$EndSheet
-$Sheet
 S 5200 4450 650  400
 U 5ED666AD
@@
 	4550 4000 4400 4000
 $Sheet
-S 5200 1700 700  1050
-U 5F099163
-F0 "LSM9DS1" 50
-F1 "LSM9DS1.sch" 50
-F2 "LSM_SCK" I L 5200 2000 50
-F3 "LSM_INT1" O L 5200 2350 50
-F4 "LSM_INT2" O L 5200 2450 50
-F5 "LSM_DEN" I L 5200 2250 50
-F6 "LSM_nCS" I L 5200 2100 50
-F7 "LSM_INT_M" O L 5200 2550 50
-F8 "LSM_DRDY_M" O L 5200 2650 50
-F9 "LSM_MOSI" I L 5200 1800 50
-F10 "LSM_MISO" O L 5200 1900 50
-$EndSheet
-$Sheet
-S 5200 3750 650  500
+S 5200 3400 700  850
 U 5EF65A4D
 F0 "BARO" 50
 F1 "BARO.sch" 50
+F2 "BARO_VIN" I L 5200 4050 50
+F3 "BARO_MOSI" I L 5200 3500 50
+F4 "BARO_MISO" O L 5200 3600 50
+F5 "BARO_SCK" I L 5200 3700 50
+F6 "BARO_MS_nCS" I L 5200 3800 50
+F7 "BARO_BMP_nCS" I L 5200 3900 50
+F8 "BARO_GND" I L 5200 4150 50
 $EndSheet
 $Comp
@@
 $EndSheet
 $Sheet
-S 5200 7200 900  400
+S 1500 7900 900  400
 U 5EF28018
 F0 "POWER_CONN" 50
 F1 "POWER_CONN.sch" 50
-F2 "BAT_CUR_SENS" O R 6100 7300 50
-F3 "BAT_VOLT_SENS" O R 6100 7400 50
-F4 "PWR_CONN_+5V" O R 6100 7500 50
-$EndSheet
-$Sheet
-S 5200 7800 900  400
+F2 "BAT_CUR_SENS" O R 2400 8100 50
+F3 "BAT_VOLT_SENS" O R 2400 8200 50
+F4 "PWR_CONN_+5V" O R 2400 8000 50
+$EndSheet
+$Sheet
+S 4400 7900 900  400
 U 5EDADA57
 F0 "MIC5504" 50
 F1 "MIC5504.sch" 50
-F2 "MIC_EN" I L 5200 8000 50
-F3 "MIC_VIN" I L 5200 7900 50
-F4 "MIC_VOUT" I R 6100 7900 50
-F5 "MIC_GND" I L 5200 8100 50
-$EndSheet
-$Sheet
-S 3050 7900 1150 450
+F2 "MIC_EN" I L 4400 8100 50
+F3 "MIC_VIN" I L 4400 8000 50
+F4 "MIC_VOUT" I R 5300 8000 50
+F5 "MIC_GND" I L 4400 8200 50
+$EndSheet
+$Sheet
+S 3050 7900 900  400
 U 5EDDEA36
 F0 "BQ24313" 50
 F1 "BQ24313.sch" 50
+F2 "BQ_IN" I L 3050 8000 50
+F3 "BQ_VSS" I L 3050 8100 50
+F4 "BQ_nFAULT" O R 3950 8100 50
+F5 "BQ_OUT" O R 3950 8000 50
+F6 "BQ_nCE" O R 3950 8200 50
+$EndSheet
+Wire Wire Line
+	2400 8000 3050 8000
+$Comp
+L power:GNDD #PWR0106
+U 1 1 5EDEC12D
+P 2950 8350
+F 0 "#PWR0106" H 2950 8100 50  0001 C CNN
+F 1 "GNDD" H 2954 8195 50  0000 C CNN
+F 2 "" H 2950 8350 50  0001 C CNN
+F 3 "" H 2950 8350 50  0001 C CNN
+	1    2950 8350
+	1    0    0    -1
+$EndComp
+Wire Wire Line
+	3050 8100 2950 8100
+Wire Wire Line
+	2950 8100 2950 8350
+Wire Wire Line
+	3950 8000 4400 8000
+$Sheet
+S 5200 1900 700  1200
+U 5EE06F22
+F0 "IMU" 50
+F1 "IMU.sch" 50
+F2 "IMU_VIN" I L 5200 2900 50
+F3 "IMU_GND" I L 5200 3000 50
+F4 "IMU_MOSI" I L 5200 2000 50
+F5 "IMU_MISO" O L 5200 2100 50
+F6 "IMU_SCK" I L 5200 2200 50
+F7 "LSM_nCS" I L 5200 2350 50
+F8 "MPU_nCS" I L 5200 2500 50
+F9 "ICM_nCS" I L 5200 2750 50
+F10 "MPU_INT" I L 5200 2600 50
 $EndSheet
 $EndSCHEMATC

Commit message: Commit
Connections:
- net labels added: CUR_SENS, VOLT_SENS
- wire segments 12 -> 69
Other:
- moved on the sheet: L5, L6, L7, L8

Commit message: Commit...
Parts:
- removed Q1: DMG2302U, Package_TO_SOT_SMD:SOT-23, symbol Transistor_FET:DMG2302U
Connections:
- net labels added: SCL1, SDA1, UART_CTS, UART_RTS, UART_RX, UART_TX
Changed lines of the file:
@@
 F8 "BARO_GND" I L 5200 4150 50
 $EndSheet
-$Comp
-L Transistor_FET:DMG2302U Q1
-U 1 1 5EFE11F6
-P 2400 1700
-F 0 "Q1" V 2742 1700 50  0000 C CNN
-F 1 "DMG2302U" V 2651 1700 50  0000 C CNN
-F 2 "Package_TO_SOT_SMD:SOT-23" H 2600 1625 50  0001 L CIN
-F 3 "http://www.diodes.com/assets/Datasheets/DMG2302U.pdf" H 2400 1700 50  0001 L CNN
-	1    2400 1700
-	0    -1   -1   0
-$EndComp
 $Sheet
 S 2150 2450 750  2750
@@
 F2 "UART_TX" O R 2900 2550 50
 F3 "UART_RX" I R 2900 2650 50
-F4 "SDA1" B R 2900 3000 50
-F5 "SCL1" O R 2900 3100 50
+F4 "SDA1" B R 2900 3100 50
+F5 "SCL1" O R 2900 3000 50
 F6 "SPI0_MOSI" O R 2900 3500 50
 F7 "SPI0_MISO" I R 2900 3600 50
@@
 F2 "GPS_TX" I L 5200 6600 50
 F3 "GPS_RX" O L 5200 6700 50
-F4 "GPS_CTS" B L 5200 6800 50
-F5 "GPS_RTS" B L 5200 6900 50
+F4 "GPS_CTS" B L 5200 6900 50
+F5 "GPS_RTS" B L 5200 6800 50
 $EndSheet
 $Sheet
@@
 	5200 4750 5000 4750
 Wire Wire Line
-	5200 6600 5000 6600
-Wire Wire Line
-	5200 6700 5000 6700
-Wire Wire Line
-	5200 6800 5000 6800
-Wire Wire Line
-	5200 6900 5000 6900
-Wire Wire Line
 	5200 6100 5000 6100
 Wire Wire Line
@@
 	4700 5500 5200 5500
 Wire Wire Line
-	2900 2550 3200 2550
-Wire Wire Line
-	2900 2650 3200 2650
-Wire Wire Line
-	2900 2750 3200 2750
-Wire Wire Line
-	2900 2850 3200 2850
-Wire Wire Line
-	2900 3000 3200 3000
-Wire Wire Line
-	2900 3100 3200 3100
-Wire Wire Line
-	2900 3250 3200 3250
-Wire Wire Line
-	2900 3350 3200 3350
-Wire Wire Line
-	2900 3500 3200 3500
-Wire Wire Line
-	2900 3600 3200 3600
-Wire Wire Line
-	2900 3700 3200 3700
-Wire Wire Line
-	2900 3800 3200 3800
-Wire Wire Line
-	2900 3950 3200 3950
-Wire Wire Line
-	2900 4050 3200 4050
-Wire Wire Line
-	2900 4150 3200 4150
-Wire Wire Line
-	2900 4250 3200 4250
+	2900 2550 3350 2550
+Wire Wire Line
+	2900 2650 3350 2650
+Wire Wire Line
+	2900 2750 3350 2750
+Wire Wire Line
+	2900 2850 3350 2850
+Wire Wire Line
+	2900 3000 3350 3000
+Wire Wire Line
+	2900 3100 3350 3100
+Wire Wire Line
+	2900 3250 3350 3250
+Wire Wire Line
+	2900 3350 3350 3350
+Wire Wire Line
+	2900 3500 3350 3500
+Wire Wire Line
+	2900 3600 3350 3600
+Wire Wire Line
+	2900 3700 3350 3700
+Wire Wire Line
+	2900 3800 3350 3800
+Wire Wire Line
+	2900 3950 3350 3950
+Wire Wire Line
+	2900 4050 3350 4050
+Wire Wire Line
+	2900 4150 3350 4150
+Wire Wire Line
+	2900 4250 3350 4250
+Text Label 3350 2550 2    50   ~ 0
+UART_TX
+Text Label 3350 2650 2    50   ~ 0
+UART_RX
+Text Label 3350 2750 2    50   ~ 0
+UART_RTS
+Text Label 3350 2850 2    50   ~ 0
+UART_CTS
+Text Label 4750 6600 0    50   ~ 0
+UART_TX
+Text Label 4750 6700 0    50   ~ 0
+UART_RX
+Text Label 4750 6800 0    50   ~ 0
+UART_RTS
+Text Label 4750 6900 0    50   ~ 0
+UART_CTS
+Wire Wire Line
+	4750 6600 5200 6600
+Wire Wire Line
+	4750 6700 5200 6700
+Wire Wire Line
+	4750 6800 5200 6800
+Wire Wire Line
+	4750 6900 5200 6900
+Text Label 3350 3100 2    50   ~ 0
+SDA1
+Text Label 3350 3000 2    50   ~ 0
+SCL1
 $EndSCHEMATC

Commit message: Commit
Connections:
- wire segments 69 -> 67
Changed lines of the file:
@@
 	4700 8000 5200 8000
 $Sheet
-S 5200 1200 550  2000
+S 5200 1200 550  1750
 U 5EE06F22
 F0 "IMU" 50
 F1 "IMU.sch" 50
-F2 "IMU_VIN" I L 5200 3000 50
-F3 "IMU_GND" I L 5200 3100 50
+F2 "IMU_VIN" I L 5200 2750 50
+F3 "IMU_GND" I L 5200 2850 50
 F4 "IMU_MOSI" I L 5200 1300 50
 F5 "IMU_MISO" O L 5200 1400 50
 F6 "IMU_SCK" I L 5200 1500 50
 F7 "LSM_nCS" I L 5200 1650 50
-F8 "MPU_nCS" I L 5200 1800 50
-F9 "ICM_nCS" I L 5200 2050 50
-F10 "MPU_INT" I L 5200 1900 50
-F11 "ICM_INT1" O L 5200 2150 50
-F12 "ICM_INT2" O L 5200 2250 50
-F13 "LSM_DEN" O L 5200 2350 50
-F14 "LSM_INT1" O L 5200 2450 50
-F15 "LSM_INT2" O L 5200 2550 50
-F16 "LSM_INT3" O L 5200 2650 50
-F17 "LSM_INT4" O L 5200 2750 50
-F18 "SENS_EN" I L 5200 2900 50
+F8 "ICM_nCS" I L 5200 1800 50
+F9 "ICM_INT1" O L 5200 1900 50
+F10 "ICM_INT2" O L 5200 2000 50
+F11 "LSM_DEN" O L 5200 2100 50
+F12 "LSM_INT1" O L 5200 2200 50
+F13 "LSM_INT2" O L 5200 2300 50
+F14 "LSM_INT3" O L 5200 2400 50
+F15 "LSM_INT4" O L 5200 2500 50
+F16 "SENS_EN" I L 5200 2650 50
 $EndSheet
 Wire Wire Line
@@
 	5200 1900 5000 1900
 Wire Wire Line
-	5200 2050 5000 2050
+	5200 2000 5000 2000
 Wire Wire Line
-	5200 2150 5000 2150
+	5200 2100 5000 2100
 Wire Wire Line
-	5200 2250 5000 2250
+	5200 2200 5000 2200
 Wire Wire Line
-	5200 2350 5000 2350
+	5200 2300 5000 2300
 Wire Wire Line
-	5200 2450 5000 2450
+	5200 2400 5000 2400
 Wire Wire Line
-	5200 2550 5000 2550
+	5200 2500 5000 2500
 Wire Wire Line
 	5200 2650 5000 2650
@@
 	5200 2750 5000 2750
 Wire Wire Line
-	5200 2900 5000 2900
-Wire Wire Line
-	5200 3000 5000 3000
-Wire Wire Line
-	5200 3100 5000 3100
+	5200 2850 5000 2850
 Wire Wire Line
 	5200 3500 5000 3500

Commit message: Commit
Connections:
- net labels added: SENS_FGND, SENS_VDD
- wire segments 67 -> 69
Changed lines of the file:
@@
 	4350 4050 4200 4050
 $Sheet
-S 5200 3400 700  850
+S 5200 2700 700  850
 U 5EF65A4D
 F0 "BARO" 50
 F1 "BARO.sch" 50
-F2 "BARO_VIN" I L 5200 4050 50
-F3 "BARO_MOSI" I L 5200 3500 50
-F4 "BARO_MISO" O L 5200 3600 50
-F5 "BARO_SCK" I L 5200 3700 50
-F6 "BARO_MS_nCS" I L 5200 3800 50
-F7 "BARO_BMP_nCS" I L 5200 3900 50
-F8 "BARO_GND" I L 5200 4150 50
+F2 "BARO_VIN" I L 5200 3350 50
+F3 "BARO_MOSI" I L 5200 2800 50
+F4 "BARO_MISO" O L 5200 2900 50
+F5 "BARO_SCK" I L 5200 3000 50
+F6 "BARO_MS_nCS" I L 5200 3100 50
+F7 "BARO_BMP_nCS" I L 5200 3200 50
+F8 "BARO_GND" I L 5200 3450 50
 $EndSheet
 $Sheet
@@
 	4700 8000 5200 8000
 $Sheet
-S 5200 1200 550  1750
+S 5200 750  550  1750
 U 5EE06F22
 F0 "IMU" 50
 F1 "IMU.sch" 50
-F2 "IMU_VIN" I L 5200 2750 50
-F3 "IMU_GND" I L 5200 2850 50
-F4 "IMU_MOSI" I L 5200 1300 50
-F5 "IMU_MISO" O L 5200 1400 50
-F6 "IMU_SCK" I L 5200 1500 50
-F7 "LSM_nCS" I L 5200 1650 50
-F8 "ICM_nCS" I L 5200 1800 50
-F9 "ICM_INT1" O L 5200 1900 50
-F10 "ICM_INT2" O L 5200 2000 50
-F11 "LSM_DEN" O L 5200 2100 50
-F12 "LSM_INT1" O L 5200 2200 50
-F13 "LSM_INT2" O L 5200 2300 50
-F14 "LSM_INT3" O L 5200 2400 50
-F15 "LSM_INT4" O L 5200 2500 50
-F16 "SENS_EN" I L 5200 2650 50
-$EndSheet
-Wire Wire Line
-	5200 1300 5000 1300
-Wire Wire Line
-	5200 1400 5000 1400
-Wire Wire Line
-	5200 1500 5000 1500
+F2 "IMU_VIN" I L 5200 2300 50
+F3 "IMU_GND" I L 5200 2400 50
+F4 "IMU_MOSI" I L 5200 850 50
+F5 "IMU_MISO" O L 5200 950 50
+F6 "IMU_SCK" I L 5200 1050 50
+F7 "LSM_nCS" I L 5200 1200 50
+F8 "ICM_nCS" I L 5200 1350 50
+F9 "ICM_INT1" O L 5200 1450 50
+F10 "ICM_INT2" O L 5200 1550 50
+F11 "LSM_DEN" O L 5200 1650 50
+F12 "LSM_INT1" O L 5200 1750 50
+F13 "LSM_INT2" O L 5200 1850 50
+F14 "LSM_INT3" O L 5200 1950 50
+F15 "LSM_INT4" O L 5200 2050 50
+F16 "SENS_EN" I L 5200 2200 50
+$EndSheet
+Wire Wire Line
+	5200 850  5000 850
+Wire Wire Line
+	5200 950  5000 950
+Wire Wire Line
+	5200 1050 5000 1050
+Wire Wire Line
+	5200 1200 5000 1200
+Wire Wire Line
+	5200 1350 5000 1350
+Wire Wire Line
+	5200 1450 5000 1450
+Wire Wire Line
+	5200 1550 5000 1550
 Wire Wire Line
 	5200 1650 5000 1650
 Wire Wire Line
-	5200 1800 5000 1800
-Wire Wire Line
-	5200 1900 5000 1900
-Wire Wire Line
-	5200 2000 5000 2000
-Wire Wire Line
-	5200 2100 5000 2100
+	5200 1750 5000 1750
+Wire Wire Line
+	5200 1850 5000 1850
+Wire Wire Line
+	5200 1950 5000 1950
+Wire Wire Line
+	5200 2050 5000 2050
 Wire Wire Line
 	5200 2200 5000 2200
 Wire Wire Line
-	5200 2300 5000 2300
-Wire Wire Line
-	5200 2400 5000 2400
-Wire Wire Line
-	5200 2500 5000 2500
-Wire Wire Line
-	5200 2650 5000 2650
-Wire Wire Line
-	5200 2750 5000 2750
-Wire Wire Line
-	5200 2850 5000 2850
-Wire Wire Line
-	5200 3500 5000 3500
-Wire Wire Line
-	5200 3600 5000 3600
-Wire Wire Line
-	5200 3700 5000 3700
-Wire Wire Line
-	5200 3800 5000 3800
-Wire Wire Line
-	5200 3900 5000 3900
-Wire Wire Line
-	5200 4050 5000 4050
-Wire Wire Line
-	5200 4150 5000 4150
+	5200 2300 4750 2300
+Wire Wire Line
+	5200 2400 4750 2400
+Wire Wire Line
+	5200 2800 5000 2800
+Wire Wire Line
+	5200 2900 5000 2900
+Wire Wire Line
+	5200 3000 5000 3000
+Wire Wire Line
+	5200 3100 5000 3100
+Wire Wire Line
+	5200 3200 5000 3200
+Wire Wire Line
+	5200 3350 4750 3350
 Wire Wire Line
 	5200 4550 5000 4550
@@
 Text Label 3350 3000 2    50   ~ 0
 SCL1
+$Sheet
+S 5200 3750 1000 400
+U 5EE7A13E
+F0 "SENSORS_POWER" 50
+F1 "SENSORS_POWER.sch" 50
+F2 "SENS_VIN" I L 5200 3850 50
+F3 "SENS_GND" I L 5200 3950 50
+F4 "SENS_EN" I L 5200 4050 50
+F5 "SENS_VDD" O R 6200 3850 50
+F6 "SENS_FGND" O R 6200 3950 50
+$EndSheet
+Wire Wire Line
+	6200 3850 6700 3850
+Text Label 6700 3850 2    50   ~ 0
+SENS_VDD
+Text Label 4750 2300 0    50   ~ 0
+SENS_VDD
+Text Label 4750 3350 0    50   ~ 0
+SENS_VDD
+Wire Wire Line
+	6200 3950 6700 3950
+Text Label 6700 3950 2    50   ~ 0
+SENS_FGND
+Text Label 4750 2400 0    50   ~ 0
+SENS_FGND
+Wire Wire Line
+	5200 3450 4750 3450
+Text Label 4750 3450 0    50   ~ 0
+SENS_FGND
 $EndSCHEMATC

Commit message: Commit
Changed lines of the file:
@@
 	5200 3200 5000 3200
 Wire Wire Line
-	5200 3350 4750 3350
-Wire Wire Line
-	5200 4550 5000 4550
-Wire Wire Line
-	5200 4650 5000 4650
+	5200 3350 4700 3350
 Wire Wire Line
 	5200 4750 5000 4750
-Wire Wire Line
-	5200 6100 5000 6100
-Wire Wire Line
-	5200 6200 5000 6200
 Wire Wire Line
 	5200 5150 5000 5150
@@
 Text Label 3350 2850 2    50   ~ 0
 UART_CTS
-Text Label 4750 6600 0    50   ~ 0
+Text Label 4700 6600 0    50   ~ 0
 UART_TX
-Text Label 4750 6700 0    50   ~ 0
+Text Label 4700 6700 0    50   ~ 0
 UART_RX
-Text Label 4750 6800 0    50   ~ 0
+Text Label 4700 6800 0    50   ~ 0
 UART_RTS
-Text Label 4750 6900 0    50   ~ 0
+Text Label 4700 6900 0    50   ~ 0
 UART_CTS
 Wire Wire Line
-	4750 6600 5200 6600
+	4700 6600 5200 6600
 Wire Wire Line
-	4750 6700 5200 6700
+	4700 6700 5200 6700
 Wire Wire Line
-	4750 6800 5200 6800
+	4700 6800 5200 6800
 Wire Wire Line
-	4750 6900 5200 6900
+	4700 6900 5200 6900
 Text Label 3350 3100 2    50   ~ 0
 SDA1
@@
 Text Label 4750 2300 0    50   ~ 0
 SENS_VDD
-Text Label 4750 3350 0    50   ~ 0
+Text Label 4700 3350 0    50   ~ 0
 SENS_VDD
 Wire Wire Line
@@
 SENS_FGND
 Wire Wire Line
-	5200 3450 4750 3450
-Text Label 4750 3450 0    50   ~ 0
+	5200 3450 4700 3450
+Text Label 4700 3450 0    50   ~ 0
 SENS_FGND
+Text Label 4700 6200 0    50   ~ 0
+SDA1
+Text Label 4700 6100 0    50   ~ 0
+SCL1
+Wire Wire Line
+	4700 6100 5200 6100
+Wire Wire Line
+	4700 6200 5200 6200
+Text Label 4700 4650 0    50   ~ 0
+SDA1
+Text Label 4700 4550 0    50   ~ 0
+SCL1
+Wire Wire Line
+	4700 4550 5200 4550
+Wire Wire Line
+	4700 4650 5200 4650
 $EndSCHEMATC

Commit message: Some changes in Sch & PCB
Parts:
- removed L5, L6, L7, L8: Ferrite_Bead, Inductor_SMD:L_0603_1608Metric, symbol Device:Ferrite_Bead
Connections:
- net labels added: SENS_MISO, SENS_MOSI, SENS_SCK, SPI0_MISO, SPI0_MOSI, SPI0_SCK
- wire segments 69 -> 66
Changed lines of the file:
@@
 $Descr A4 8268 11693 portrait
 encoding utf-8
-Sheet 1 17
+Sheet 1 18
 Title "RasPi Zero NAV Hat"
-Date "2020-06-08"
+Date "2020-08-11"
 Rev "0.1"
 Comp "chipiki.ru"
@@
 F4 "PCA_nOE" I L 5200 4750 50
 $EndSheet
-$Comp
-L Device:Ferrite_Bead L?
-U 1 1 5ED6AF36
-P 4050 3150
-AR Path="/5ED65008/5ED6AF36" Ref="L?"  Part="1"
-AR Path="/5ED6AF36" Ref="L5"  Part="1"
-F 0 "L5" V 4100 3250 50  0000 C CNN
-F 1 "Ferrite_Bead" V 3600 3150 50  0000 C CNN
-F 2 "Inductor_SMD:L_0603_1608Metric" V 3980 3150 50  0001 C CNN
-F 3 "~" H 4050 3150 50  0001 C CNN
-	1    4050 3150
-	0    1    -1   0
-$EndComp
-Wire Wire Line
-	3900 3150 3750 3150
-$Comp
-L Device:Ferrite_Bead L?
-U 1 1 5ED6B9DB
-P 4050 3450
-AR Path="/5ED65008/5ED6B9DB" Ref="L?"  Part="1"
-AR Path="/5ED6B9DB" Ref="L6"  Part="1"
-F 0 "L6" V 4100 3550 50  0000 C CNN
-F 1 "Ferrite_Bead" V 4200 3450 50  0000 C CNN
-F 2 "Inductor_SMD:L_0603_1608Metric" V 3980 3450 50  0001 C CNN
-F 3 "~" H 4050 3450 50  0001 C CNN
-	1    4050 3450
-	0    1    -1   0
-$EndComp
-Wire Wire Line
-	3900 3450 3750 3450
-$Comp
-L Device:Ferrite_Bead L?
-U 1 1 5ED6CB61
-P 4050 3750
-AR Path="/5ED65008/5ED6CB61" Ref="L?"  Part="1"
-AR Path="/5ED6CB61" Ref="L7"  Part="1"
-F 0 "L7" V 4100 3850 50  0000 C CNN
-F 1 "Ferrite_Bead" V 3600 3750 50  0000 C CNN
-F 2 "Inductor_SMD:L_0603_1608Metric" V 3980 3750 50  0001 C CNN
-F 3 "~" H 4050 3750 50  0001 C CNN
-	1    4050 3750
-	0    1    -1   0
-$EndComp
-Wire Wire Line
-	3900 3750 3750 3750
-$Comp
-L Device:Ferrite_Bead L?
-U 1 1 5ED6CB68
-P 4050 4050
-AR Path="/5ED65008/5ED6CB68" Ref="L?"  Part="1"
-AR Path="/5ED6CB68" Ref="L8"  Part="1"
-F 0 "L8" V 4100 4150 50  0000 C CNN
-F 1 "Ferrite_Bead" V 4200 4050 50  0000 C CNN
-F 2 "Inductor_SMD:L_0603_1608Metric" V 3980 4050 50  0001 C CNN
-F 3 "~" H 4050 4050 50  0001 C CNN
-	1    4050 4050
-	0    1    -1   0
-$EndComp
-Wire Wire Line
-	3900 4050 3750 4050
-Wire Wire Line
-	4350 3150 4200 3150
-Wire Wire Line
-	4350 3450 4200 3450
-Wire Wire Line
-	4350 3750 4200 3750
-Wire Wire Line
-	4350 4050 4200 4050
 $Sheet
 S 5200 2700 700  850
@@
 F2 "IMU_VIN" I L 5200 2300 50
 F3 "IMU_GND" I L 5200 2400 50
-F4 "IMU_MOSI" I L 5200 850 50
-F5 "IMU_MISO" O L 5200 950 50
-F6 "IMU_SCK" I L 5200 1050 50
-F7 "LSM_nCS" I L 5200 1200 50
-F8 "ICM_nCS" I L 5200 1350 50
-F9 "ICM_INT1" O L 5200 1450 50
-F10 "ICM_INT2" O L 5200 1550 50
-F11 "LSM_DEN" O L 5200 1650 50
-F12 "LSM_INT1" O L 5200 1750 50
-F13 "LSM_INT2" O L 5200 1850 50
-F14 "LSM_INT3" O L 5200 1950 50
-F15 "LSM_INT4" O L 5200 2050 50
-F16 "SENS_EN" I L 5200 2200 50
-$EndSheet
-Wire Wire Line
-	5200 850  5000 850
-Wire Wire Line
-	5200 950  5000 950
-Wire Wire Line
-	5200 1050 5000 1050
-Wire Wire Line
-	5200 1200 5000 1200
-Wire Wire Line
-	5200 1350 5000 1350
-Wire Wire Line
-	5200 1450 5000 1450
-Wire Wire Line
-	5200 1550 5000 1550
-Wire Wire Line
-	5200 1650 5000 1650
-Wire Wire Line
-	5200 1750 5000 1750
-Wire Wire Line
-	5200 1850 5000 1850
-Wire Wire Line
-	5200 1950 5000 1950
-Wire Wire Line
-	5200 2050 5000 2050
-Wire Wire Line
-	5200 2200 5000 2200
+F4 "LSM_nCS" I L 5200 1200 50
+F5 "ICM_nCS" I L 5200 1300 50
+F6 "ICM_INT1" O L 5200 1450 50
+F7 "ICM_INT2" O L 5200 1550 50
+F8 "LSM_DEN" O L 5200 1650 50
+F9 "LSM_INT1" O L 5200 1750 50
+F10 "LSM_INT2" O L 5200 1850 50
+F11 "LSM_INT3" O L 5200 1950 50
+F12 "LSM_INT4" O L 5200 2050 50
+F13 "IMU_MOSI" I L 5200 850 50
+F14 "IMU_MISO" O L 5200 950 50
+F15 "IMU_SCK" I L 5200 1050 50
+$EndSheet
+Wire Wire Line
+	5200 850  4750 850
+Wire Wire Line
+	5200 950  4750 950
+Wire Wire Line
+	5200 1050 4750 1050
+Wire Wire Line
+	5200 1200 4750 1200
+Wire Wire Line
+	5200 1300 4750 1300
+Wire Wire Line
+	5200 1450 4750 1450
+Wire Wire Line
+	5200 1550 4750 1550
+Wire Wire Line
+	5200 1650 4750 1650
+Wire Wire Line
+	5200 1750 4750 1750
+Wire Wire Line
+	5200 1850 4750 1850
+Wire Wire Line
+	5200 1950 4750 1950
+Wire Wire Line
+	5200 2050 4750 2050
 Wire Wire Line
 	5200 2300 4750 2300
@@
 Wire Wire Line
 	5200 4750 5000 4750
-Wire Wire Line
-	5200 5150 5000 5150
-Wire Wire Line
-	5200 5250 5000 5250
 Wire Wire Line
 	5200 5600 5000 5600
@@
 Wire Wire Line
 	2900 3350 3350 3350
-Wire Wire Line
-	2900 3500 3350 3500
-Wire Wire Line
-	2900 3600 3350 3600
-Wire Wire Line
-	2900 3700 3350 3700
 Wire Wire Line
 	2900 3800 3350 3800
@@
 Wire Wire Line
 	4700 4650 5200 4650
+Text Label 4700 5250 0    50   ~ 0
+SDA1
+Text Label 4700 5150 0    50   ~ 0
+SCL1
+Wire Wire Line
+	4700 5150 5200 5150
+Wire Wire Line
+	4700 5250 5200 5250
+Text Label 4750 850  0    50   ~ 0
+SENS_MOSI
+Text Label 4750 950  0    50   ~ 0
+SENS_MISO
+Text Label 4750 1050 0    50   ~ 0
+SENS_SCK
+$Sheet
+S 2350 6050 800  500
+U 5F329359
+F0 "FB" 50
+F1 "FerriteBeads.sch" 50
+F2 "X1" U L 2350 6150 50
+F3 "X2" U L 2350 6250 50
+F4 "X3" U L 2350 6350 50
+F5 "X4" U L 2350 6450 50
+F6 "Y1" U R 3150 6150 50
+F7 "Y2" U R 3150 6250 50
+F8 "Y3" U R 3150 6350 50
+F9 "Y4" U R 3150 6450 50
+$EndSheet
+Wire Wire Line
+	3150 6150 3600 6150
+Wire Wire Line
+	3150 6250 3600 6250
+Wire Wire Line
+	3150 6350 3600 6350
+Text Label 3600 6150 2    50   ~ 0
+SENS_MOSI
+Text Label 3600 6250 2    50   ~ 0
+SENS_MISO
+Text Label 3600 6350 2    50   ~ 0
+SENS_SCK
+Text Label 3350 3500 2    50   ~ 0
+SPI0_MOSI
+Text Label 3350 3600 2    50   ~ 0
+SPI0_MISO
+Text Label 3350 3700 2    50   ~ 0
+SPI0_SCK
+Wire Wire Line
+	2350 6150 1900 6150
+Wire Wire Line
+	2350 6250 1900 6250
+Wire Wire Line
+	2350 6350 1900 6350
+Text Label 1900 6150 0    50   ~ 0
+SPI0_MOSI
+Text Label 1900 6250 0    50   ~ 0
+SPI0_MISO
+Text Label 1900 6350 0    50   ~ 0
+SPI0_SCK
+Wire Wire Line
+	2900 3500 3350 3500
+Wire Wire Line
+	2900 3600 3350 3600
+Wire Wire Line
+	2900 3700 3350 3700
 $EndSCHEMATC
