File: HW/rbpi-z-hat/ADS1015.sch (KiCad schematic (older format))
At the start: 6 parts

Commit message: Commit...
Parts:
- C6: renamed from C?; footprint (none) -> Capacitor_SMD:C_0603_1608Metric
- gave numbers to parts that had none: 5
Changed lines of the file:
@@
 $Descr A4 8268 11693 portrait
 encoding utf-8
-Sheet 11 14
+Sheet 10 18
 Title "RasPi Zero NAV Hat"
 Date "2020-06-08"
@@
 P 4550 5500
 AR Path="/5EF08EAF" Ref="U?"  Part="1"
-AR Path="/5EF0850C/5EF08EAF" Ref="U?"  Part="1"
-F 0 "U?" H 4300 5950 50  0000 C CNN
+AR Path="/5EF0850C/5EF08EAF" Ref="U6"  Part="1"
+F 0 "U6" H 4300 5950 50  0000 C CNN
 F 1 "ADS1015IDGS" H 4850 5150 50  0000 C CNN
 F 2 "Package_SO:TSSOP-10_3x3mm_P0.5mm" H 4550 5000 50  0001 C CNN
@@
 Connection ~ 4550 5950
 $Comp
-L Device:C C?
+L Device:C C6
 U 1 1 5EF0AD07
 P 4800 4800
-F 0 "C?" V 4548 4800 50  0000 C CNN
+F 0 "C6" V 4548 4800 50  0000 C CNN
 F 1 "0.1uF" V 4639 4800 50  0000 C CNN
-F 2 "" H 4838 4650 50  0001 C CNN
+F 2 "Capacitor_SMD:C_0603_1608Metric" H 4838 4650 50  0001 C CNN
 F 3 "~" H 4800 4800 50  0001 C CNN
 	1    4800 4800
@@
 P 5000 4900
 AR Path="/5EDD13AE/5EF0CA1D" Ref="#PWR?"  Part="1"
-AR Path="/5EF0850C/5EF0CA1D" Ref="#PWR?"  Part="1"
-F 0 "#PWR?" H 5000 4650 50  0001 C CNN
+AR Path="/5EF0850C/5EF0CA1D" Ref="#PWR0135"  Part="1"
+F 0 "#PWR0135" H 5000 4650 50  0001 C CNN
 F 1 "GNDD" H 5004 4745 50  0000 C CNN
 F 2 "" H 5000 4900 50  0001 C CNN
@@
 AR Path="/5EF65A4D/5EF663FB/5EDA4EF4" Ref="L?"  Part="1"
 AR Path="/5EF65A4D/5EDA4EF4" Ref="L?"  Part="1"
-AR Path="/5EF0850C/5EDA4EF4" Ref="L?"  Part="1"
-F 0 "L?" V 4750 7250 50  0000 C CNN
+AR Path="/5EF0850C/5EDA4EF4" Ref="L1"  Part="1"
+F 0 "L1" V 4750 7250 50  0000 C CNN
 F 1 "Ferrite_Bead" V 4650 7250 50  0000 C CNN
 F 2 "Inductor_SMD:L_0603_1608Metric" V 4430 7250 50  0001 C CNN
@@
 AR Path="/5EF65A4D/5EF663FB/5EDA4EFA" Ref="C?"  Part="1"
 AR Path="/5EF65A4D/5EDA4EFA" Ref="C?"  Part="1"
-AR Path="/5EF0850C/5EDA4EFA" Ref="C?"  Part="1"
-F 0 "C?" H 4300 7900 50  0000 L CNN
+AR Path="/5EF0850C/5EDA4EFA" Ref="C7"  Part="1"
+F 0 "C7" H 4300 7900 50  0000 L CNN
 F 1 "100nF" H 4300 7700 50  0000 L CNN
 F 2 "Capacitor_SMD:C_0603_1608Metric" H 4288 7650 50  0001 C CNN
@@
 AR Path="/5EF65A4D/5EF663FB/5EDA4F04" Ref="#PWR?"  Part="1"
 AR Path="/5EF65A4D/5EDA4F04" Ref="#PWR?"  Part="1"
-AR Path="/5EF0850C/5EDA4F04" Ref="#PWR?"  Part="1"
-F 0 "#PWR?" H 4250 8250 50  0001 C CNN
+AR Path="/5EF0850C/5EDA4F04" Ref="#PWR0136"  Part="1"
+F 0 "#PWR0136" H 4250 8250 50  0001 C CNN
 F 1 "GNDD" H 4254 8345 50  0000 C CNN
 F 2 "" H 4250 8500 50  0001 C CNN
@@
 AR Path="/5EF65A4D/5EF663FB/5EDA4F0C" Ref="L?"  Part="1"
 AR Path="/5EF65A4D/5EDA4F0C" Ref="L?"  Part="1"
-AR Path="/5EF0850C/5EDA4F0C" Ref="L?"  Part="1"
-F 0 "L?" V 4700 8350 50  0000 C CNN
+AR Path="/5EF0850C/5EDA4F0C" Ref="L4"  Part="1"
+F 0 "L4" V 4700 8350 50  0000 C CNN
 F 1 "Ferrite_Bead" V 4350 8350 50  0000 C CNN
 F 2 "Inductor_SMD:L_0603_1608Metric" V 4430 8350 50  0001 C CNN
@@
 AR Path="/5EF65A4D/5EF663FB/5EDA4F16" Ref="#PWR?"  Part="1"
 AR Path="/5EF65A4D/5EDA4F16" Ref="#PWR?"  Part="1"
-AR Path="/5EF0850C/5EDA4F16" Ref="#PWR?"  Part="1"
-F 0 "#PWR?" H 4250 6850 50  0001 C CNN
+AR Path="/5EF0850C/5EDA4F16" Ref="#PWR0137"  Part="1"
+F 0 "#PWR0137" H 4250 6850 50  0001 C CNN
 F 1 "+3.3V" H 4265 7173 50  0000 C CNN
 F 2 "" H 4250 7000 50  0001 C CNN
@@
 AR Path="/5EF65A4D/5EF663FB/5EDA4F1D" Ref="C?"  Part="1"
 AR Path="/5EF65A4D/5EDA4F1D" Ref="C?"  Part="1"
-AR Path="/5EF0850C/5EDA4F1D" Ref="C?"  Part="1"
-F 0 "C?" H 4700 7900 50  0000 L CNN
+AR Path="/5EF0850C/5EDA4F1D" Ref="C10"  Part="1"
+F 0 "C10" H 4700 7900 50  0000 L CNN
 F 1 "22uF/10V" H 4450 7700 50  0000 L CNN
 F 2 "Capacitor_SMD:C_1206_3216Metric" H 4888 7650 50  0001 C CNN

Commit message: Commit
Connections:
- net ADS_GND: now also C6.1
- net GNDD: no longer C6.1
Changed lines of the file:
@@
 	0    1    1    0
 $EndComp
-$Comp
-L power:GNDD #PWR?
-U 1 1 5EF0CA1D
-P 5000 4900
-AR Path="/5EDD13AE/5EF0CA1D" Ref="#PWR?"  Part="1"
-AR Path="/5EF0850C/5EF0CA1D" Ref="#PWR0135"  Part="1"
-F 0 "#PWR0135" H 5000 4650 50  0001 C CNN
-F 1 "GNDD" H 5004 4745 50  0000 C CNN
-F 2 "" H 5000 4900 50  0001 C CNN
-F 3 "" H 5000 4900 50  0001 C CNN
-	1    5000 4900
-	1    0    0    -1
-$EndComp
 Wire Wire Line
-	5000 4800 5000 4900
-Wire Wire Line
-	4950 4800 5000 4800
+	4950 4800 5350 4800
 Wire Wire Line
 	4550 5000 4550 4800
@@
 Wire Wire Line
 	4550 4450 4550 4800
+Text Label 5350 4800 2    50   ~ 0
+ADS_GND
 $EndSCHEMATC
