File: HW/rbpi-z-hat/BARO.sch (KiCad schematic (older format))
At the start: 4 parts

Commit message: Commit...
Parts:
- removed C10: 22uF/10V, Capacitor_SMD:C_1206_3216Metric, symbol Device:C
Connections:
- net GNDD is gone; now on net BARO_GND: C12.2, L3.1
- net BARO_GND: no longer L3.2
- net BARO_VDD: no longer L2.2
- net +3V3 renamed BARO_VIN
- new net BARO_FGND: L3.2
- new net MIC5504_BARO/MIC_VIN: L2.2
Other:
- note removed: "CL31B226KPHNNNE"
- moved on the sheet: C12, L2, L3
Changed lines of the file:
@@
 $Descr A4 8268 11693 portrait
 encoding utf-8
-Sheet 5 14
+Sheet 3 18
 Title "RasPi Zero NAV Hat"
 Date "2020-06-08"
@@
 $EndDescr
 $Sheet
-S 5200 4700 700  750
+S 4850 3400 700  750
 U 5EF663FB
 F0 "MS5611" 50
 F1 "MS5611.sch" 50
-F2 "MS_nCS" I L 5200 5100 50
-F3 "MS_MOSI" I L 5200 4800 50
-F4 "MS_SCK" I L 5200 5000 50
-F5 "MS_MISO" O L 5200 4900 50
-F6 "MS_VDD" U L 5200 5250 50
-F7 "MS_GND" U L 5200 5350 50
+F2 "MS_nCS" I L 4850 3800 50
+F3 "MS_MOSI" I L 4850 3500 50
+F4 "MS_SCK" I L 4850 3700 50
+F5 "MS_MISO" O L 4850 3600 50
+F6 "MS_VDD" U L 4850 3950 50
+F7 "MS_GND" U L 4850 4050 50
 $EndSheet
 $Sheet
-S 5200 5650 700  750
+S 4850 4350 700  750
 U 5EF663FD
 F0 "BMP280" 50
 F1 "BMP280.sch" 50
-F2 "BMP_SCK" I L 5200 5950 50
-F3 "BMP_MOSI" I L 5200 5750 50
-F4 "BMP_MISO" O L 5200 5850 50
-F5 "BMP_nCS" I L 5200 6050 50
-F6 "BMP_VDD" U L 5200 6200 50
-F7 "BPM_GND" U L 5200 6300 50
+F2 "BMP_SCK" I L 4850 4650 50
+F3 "BMP_MOSI" I L 4850 4450 50
+F4 "BMP_MISO" O L 4850 4550 50
+F5 "BMP_nCS" I L 4850 4750 50
+F6 "BMP_VDD" U L 4850 4900 50
+F7 "BPM_GND" U L 4850 5000 50
 $EndSheet
 Wire Wire Line
-	4250 5000 3800 5000
+	6200 6500 5750 6500
 Wire Wire Line
-	3800 5000 3800 5400
-Wire Wire Line
-	4250 6100 3800 6100
-Wire Wire Line
-	3800 6100 3800 5700
+	5300 7600 4800 7600
 $Comp
 L Device:Ferrite_Bead L?
 U 1 1 5EF7256D
-P 3450 5000
+P 4400 6500
 AR Path="/5ED663F7/5EF7256D" Ref="L?"  Part="1"
 AR Path="/5EF65A4D/5EF663FB/5EF7256D" Ref="L?"  Part="1"
 AR Path="/5EF65A4D/5EF7256D" Ref="L2"  Part="1"
-F 0 "L2" V 3700 5000 50  0000 C CNN
-F 1 "Ferrite_Bead" V 3600 5000 50  0000 C CNN
-F 2 "Inductor_SMD:L_0603_1608Metric" V 3380 5000 50  0001 C CNN
-F 3 "~" H 3450 5000 50  0001 C CNN
-	1    3450 5000
+F 0 "L2" V 4650 6500 50  0000 C CNN
+F 1 "Ferrite_Bead" V 4550 6500 50  0000 C CNN
+F 2 "Inductor_SMD:L_0603_1608Metric" V 4330 6500 50  0001 C CNN
+F 3 "~" H 4400 6500 50  0001 C CNN
+	1    4400 6500
 	0    -1   -1   0
 $EndComp
@@
 L Device:C C?
 U 1 1 5EF72573
-P 3200 5550
+P 4150 7050
 AR Path="/5ED663F7/5EF72573" Ref="C?"  Part="1"
 AR Path="/5EF65A4D/5EF663FB/5EF72573" Ref="C?"  Part="1"
 AR Path="/5EF65A4D/5EF72573" Ref="C12"  Part="1"
-F 0 "C12" H 3250 5650 50  0000 L CNN
-F 1 "100nF" H 3250 5450 50  0000 L CNN
-F 2 "Capacitor_SMD:C_0603_1608Metric" H 3238 5400 50  0001 C CNN
-F 3 "" H 3200 5550 50  0001 C CNN
-	1    3200 5550
+F 0 "C12" H 4200 7150 50  0000 L CNN
+F 1 "100nF" H 4200 6950 50  0000 L CNN
+F 2 "Capacitor_SMD:C_0603_1608Metric" H 4188 6900 50  0001 C CNN
+F 3 "" H 4150 7050 50  0001 C CNN
+	1    4150 7050
 	1    0    0    -1
 $EndComp
 Wire Wire Line
-	3200 4750 3200 5000
+	3900 6500 4150 6500
 Wire Wire Line
-	3300 5000 3200 5000
-Connection ~ 3200 5000
+	4250 6500 4150 6500
+Connection ~ 4150 6500
 Wire Wire Line
-	3200 5000 3200 5400
-$Comp
-L power:GNDD #PWR?
-U 1 1 5EF7257D
-P 3200 6250
-AR Path="/5ED663F7/5EF7257D" Ref="#PWR?"  Part="1"
-AR Path="/5EF65A4D/5EF663FB/5EF7257D" Ref="#PWR?"  Part="1"
-AR Path="/5EF65A4D/5EF7257D" Ref="#PWR0110"  Part="1"
-F 0 "#PWR0110" H 3200 6000 50  0001 C CNN
-F 1 "GNDD" H 3204 6095 50  0000 C CNN
-F 2 "" H 3200 6250 50  0001 C CNN
-F 3 "" H 3200 6250 50  0001 C CNN
-	1    3200 6250
-	1    0    0    -1
-$EndComp
-Connection ~ 3800 5000
+	4150 6500 4150 6900
 Wire Wire Line
-	3200 5700 3200 6100
+	4150 7200 4150 7600
 $Comp
 L Device:Ferrite_Bead L?
 U 1 1 5EF72585
-P 3450 6100
+P 4400 7600
 AR Path="/5ED663F7/5EF72585" Ref="L?"  Part="1"
 AR Path="/5EF65A4D/5EF663FB/5EF72585" Ref="L?"  Part="1"
 AR Path="/5EF65A4D/5EF72585" Ref="L3"  Part="1"
-F 0 "L3" V 3650 6100 50  0000 C CNN
-F 1 "Ferrite_Bead" V 3300 6100 50  0000 C CNN
-F 2 "Inductor_SMD:L_0603_1608Metric" V 3380 6100 50  0001 C CNN
-F 3 "~" H 3450 6100 50  0001 C CNN
-	1    3450 6100
+F 0 "L3" V 4600 7600 50  0000 C CNN
+F 1 "Ferrite_Bead" V 4250 7600 50  0000 C CNN
+F 2 "Inductor_SMD:L_0603_1608Metric" V 4330 7600 50  0001 C CNN
+F 3 "~" H 4400 7600 50  0001 C CNN
+	1    4400 7600
 	0    -1   -1   0
 $EndComp
 Wire Wire Line
-	3300 6100 3200 6100
-Connection ~ 3200 6100
+	4250 7600 4150 7600
+Text Label 6200 6500 2    50   ~ 0
+BARO_VDD
+Text Label 5300 7600 2    50   ~ 0
+BARO_FGND
 Wire Wire Line
-	3200 6100 3200 6250
-Connection ~ 3800 6100
-$Comp
-L power:+3.3V #PWR?
-U 1 1 5EF7258F
-P 3200 4750
-AR Path="/5ED663F7/5EF7258F" Ref="#PWR?"  Part="1"
-AR Path="/5EF65A4D/5EF663FB/5EF7258F" Ref="#PWR?"  Part="1"
-AR Path="/5EF65A4D/5EF7258F" Ref="#PWR0111"  Part="1"
-F 0 "#PWR0111" H 3200 4600 50  0001 C CNN
-F 1 "+3.3V" H 3215 4923 50  0000 C CNN
-F 2 "" H 3200 4750 50  0001 C CNN
-F 3 "" H 3200 4750 50  0001 C CNN
-	1    3200 4750
-	-1   0    0    -1
-$EndComp
-$Comp
-L Device:C C?
-U 1 1 5EF72596
-P 3800 5550
-AR Path="/5ED663F7/5EF72596" Ref="C?"  Part="1"
-AR Path="/5EF65A4D/5EF663FB/5EF72596" Ref="C?"  Part="1"
-AR Path="/5EF65A4D/5EF72596" Ref="C10"  Part="1"
-F 0 "C10" H 3650 5650 50  0000 L CNN
-F 1 "22uF/10V" H 3400 5450 50  0000 L CNN
-F 2 "Capacitor_SMD:C_1206_3216Metric" H 3838 5400 50  0001 C CNN
-F 3 "" H 3800 5550 50  0001 C CNN
-F 4 "https://www.terraelectronica.ru/product/1641498" H 3800 5550 50  0001 C CNN "URL"
-	1    3800 5550
-	-1   0    0    -1
-$EndComp
-Text Notes 3700 5950 1    50   ~ 0
-CL31B226KPHNNNE
-Wire Wire Line
-	3800 5000 3600 5000
-Wire Wire Line
-	3800 6100 3600 6100
-Text Label 4250 5000 2    50   ~ 0
-BARO_VDD
-Text Label 4250 6100 2    50   ~ 0
-BARO_GND
-Wire Wire Line
-	4750 5250 5200 5250
-Text Label 4750 5250 0    50   ~ 0
+	4350 3950 4850 3950
+Text Label 4350 3950 0    50   ~ 0
 BARO_VDD
 Wire Wire Line
-	4750 5350 5200 5350
-Text Label 4750 5350 0    50   ~ 0
-BARO_GND
+	4350 4050 4850 4050
+Text Label 4350 4050 0    50   ~ 0
+BARO_FGND
 Wire Wire Line
-	4750 6200 5200 6200
-Text Label 4750 6200 0    50   ~ 0
+	4350 4900 4850 4900
+Text Label 4350 4900 0    50   ~ 0
 BARO_VDD
 Wire Wire Line
-	4750 6300 5200 6300
-Text Label 4750 6300 0    50   ~ 0
+	4350 5000 4850 5000
+Text Label 4350 5000 0    50   ~ 0
+BARO_FGND
+$Sheet
+S 4850 6400 900  400
+U 5EE0D50D
+F0 "MIC5504_BARO" 50
+F1 "MIC5504.sch" 50
+F2 "MIC_EN" I L 4850 6600 50
+F3 "MIC_VIN" I L 4850 6500 50
+F4 "MIC_VOUT" I R 5750 6500 50
+F5 "MIC_GND" I L 4850 6700 50
+$EndSheet
+Wire Wire Line
+	4850 6700 4800 6700
+Wire Wire Line
+	4800 6700 4800 7600
+Connection ~ 4800 7600
+Wire Wire Line
+	4550 6500 4850 6500
+Wire Wire Line
+	4550 7600 4800 7600
+Wire Wire Line
+	4150 7600 3900 7600
+Connection ~ 4150 7600
+Text HLabel 3900 6500 0    50   Input ~ 0
+BARO_VIN
+Text HLabel 3450 3500 0    50   Input ~ 0
+BARO_MOSI
+Text HLabel 3450 3600 0    50   Output ~ 0
+BARO_MISO
+Text HLabel 3450 3700 0    50   Input ~ 0
+BARO_SCK
+Text HLabel 3450 3800 0    50   Input ~ 0
+BARO_MS_nCS
+Text HLabel 3400 4750 0    50   Input ~ 0
+BARO_BMP_nCS
+Wire Wire Line
+	3400 4750 4850 4750
+Wire Wire Line
+	3450 3800 4850 3800
+Wire Wire Line
+	3450 3700 4050 3700
+Wire Wire Line
+	3450 3600 4150 3600
+Wire Wire Line
+	3450 3500 4250 3500
+Wire Wire Line
+	4250 4450 4250 3500
+Wire Wire Line
+	4250 4450 4850 4450
+Connection ~ 4250 3500
+Wire Wire Line
+	4250 3500 4850 3500
+Wire Wire Line
+	4150 4550 4150 3600
+Wire Wire Line
+	4150 4550 4850 4550
+Connection ~ 4150 3600
+Wire Wire Line
+	4150 3600 4850 3600
+Wire Wire Line
+	4050 4650 4050 3700
+Wire Wire Line
+	4050 4650 4850 4650
+Connection ~ 4050 3700
+Wire Wire Line
+	4050 3700 4850 3700
+Text HLabel 3900 7600 0    50   Input ~ 0
 BARO_GND
 $EndSCHEMATC

Commit message: Commit
Parts:
- removed C12: 100nF, Capacitor_SMD:C_0603_1608Metric, symbol Device:C
- removed L2, L3: Ferrite_Bead, Inductor_SMD:L_0603_1608Metric, symbol Device:Ferrite_Bead
- added C?: 22uF/10V, Capacitor_SMD:C_1206_3216Metric, symbol Device:C
Connections:
- net BARO_GND: now also C?.2
- net BARO_VIN: now also C?.1
Other:
- note added: "CL31B226KPHNNNE"
Changed lines of the file:
@@
 $EndSheet
 Wire Wire Line
-	6200 6500 5750 6500
-Wire Wire Line
-	5300 7600 4800 7600
-$Comp
-L Device:Ferrite_Bead L?
-U 1 1 5EF7256D
-P 4400 6500
-AR Path="/5ED663F7/5EF7256D" Ref="L?"  Part="1"
-AR Path="/5EF65A4D/5EF663FB/5EF7256D" Ref="L?"  Part="1"
-AR Path="/5EF65A4D/5EF7256D" Ref="L2"  Part="1"
-F 0 "L2" V 4650 6500 50  0000 C CNN
-F 1 "Ferrite_Bead" V 4550 6500 50  0000 C CNN
-F 2 "Inductor_SMD:L_0603_1608Metric" V 4330 6500 50  0001 C CNN
-F 3 "~" H 4400 6500 50  0001 C CNN
-	1    4400 6500
-	0    -1   -1   0
-$EndComp
-$Comp
-L Device:C C?
-U 1 1 5EF72573
-P 4150 7050
-AR Path="/5ED663F7/5EF72573" Ref="C?"  Part="1"
-AR Path="/5EF65A4D/5EF663FB/5EF72573" Ref="C?"  Part="1"
-AR Path="/5EF65A4D/5EF72573" Ref="C12"  Part="1"
-F 0 "C12" H 4200 7150 50  0000 L CNN
-F 1 "100nF" H 4200 6950 50  0000 L CNN
-F 2 "Capacitor_SMD:C_0603_1608Metric" H 4188 6900 50  0001 C CNN
-F 3 "" H 4150 7050 50  0001 C CNN
-	1    4150 7050
-	1    0    0    -1
-$EndComp
-Wire Wire Line
-	3900 6500 4150 6500
-Wire Wire Line
-	4250 6500 4150 6500
-Connection ~ 4150 6500
-Wire Wire Line
-	4150 6500 4150 6900
-Wire Wire Line
-	4150 7200 4150 7600
-$Comp
-L Device:Ferrite_Bead L?
-U 1 1 5EF72585
-P 4400 7600
-AR Path="/5ED663F7/5EF72585" Ref="L?"  Part="1"
-AR Path="/5EF65A4D/5EF663FB/5EF72585" Ref="L?"  Part="1"
-AR Path="/5EF65A4D/5EF72585" Ref="L3"  Part="1"
-F 0 "L3" V 4600 7600 50  0000 C CNN
-F 1 "Ferrite_Bead" V 4250 7600 50  0000 C CNN
-F 2 "Inductor_SMD:L_0603_1608Metric" V 4330 7600 50  0001 C CNN
-F 3 "~" H 4400 7600 50  0001 C CNN
-	1    4400 7600
-	0    -1   -1   0
-$EndComp
-Wire Wire Line
-	4250 7600 4150 7600
-Text Label 6200 6500 2    50   ~ 0
-BARO_VDD
-Text Label 5300 7600 2    50   ~ 0
-BARO_FGND
+	3450 5900 3700 5900
 Wire Wire Line
 	4350 3950 4850 3950
@@
 Text Label 4350 5000 0    50   ~ 0
 BARO_FGND
-$Sheet
-S 4850 6400 900  400
-U 5EE0D50D
-F0 "MIC5504_BARO" 50
-F1 "MIC5504.sch" 50
-F2 "MIC_EN" I L 4850 6600 50
-F3 "MIC_VIN" I L 4850 6500 50
-F4 "MIC_VOUT" I R 5750 6500 50
-F5 "MIC_GND" I L 4850 6700 50
-$EndSheet
-Wire Wire Line
-	4850 6700 4800 6700
-Wire Wire Line
-	4800 6700 4800 7600
-Connection ~ 4800 7600
-Wire Wire Line
-	4550 6500 4850 6500
-Wire Wire Line
-	4550 7600 4800 7600
-Wire Wire Line
-	4150 7600 3900 7600
-Connection ~ 4150 7600
-Text HLabel 3900 6500 0    50   Input ~ 0
+Text HLabel 3450 5900 0    50   Input ~ 0
 BARO_VIN
 Text HLabel 3450 3500 0    50   Input ~ 0
@@
 Text HLabel 3450 3800 0    50   Input ~ 0
 BARO_MS_nCS
-Text HLabel 3400 4750 0    50   Input ~ 0
+Text HLabel 3450 4750 0    50   Input ~ 0
 BARO_BMP_nCS
 Wire Wire Line
-	3400 4750 4850 4750
+	3450 4750 4850 4750
 Wire Wire Line
 	3450 3800 4850 3800
@@
 Wire Wire Line
 	4050 3700 4850 3700
-Text HLabel 3900 7600 0    50   Input ~ 0
+Text HLabel 3450 6700 0    50   Input ~ 0
 BARO_GND
+Wire Wire Line
+	3700 5900 3700 6150
+Wire Wire Line
+	3700 6700 3700 6450
+$Comp
+L Device:C C?
+U 1 1 5EE69A69
+P 3700 6300
+AR Path="/5ED663F7/5EE69A69" Ref="C?"  Part="1"
+AR Path="/5EF65A4D/5EF663FB/5EE69A69" Ref="C?"  Part="1"
+AR Path="/5EF65A4D/5EE69A69" Ref="C?"  Part="1"
+AR Path="/5EDADA57/5EE69A69" Ref="C?"  Part="1"
+AR Path="/5EF65A4D/5EE0D50D/5EE69A69" Ref="C?"  Part="1"
+AR Path="/5EE06F22/5EE2A025/5EE69A69" Ref="C?"  Part="1"
+F 0 "C?" H 3550 6400 50  0000 L CNN
+F 1 "22uF/10V" H 3300 6200 50  0000 L CNN
+F 2 "Capacitor_SMD:C_1206_3216Metric" H 3738 6150 50  0001 C CNN
+F 3 "" H 3700 6300 50  0001 C CNN
+F 4 "https://www.terraelectronica.ru/product/1641498" H 3700 6300 50  0001 C CNN "URL"
+	1    3700 6300
+	-1   0    0    -1
+$EndComp
+Text Notes 3600 6700 1    50   ~ 0
+CL31B226KPHNNNE
+Wire Wire Line
+	3450 6700 3700 6700
+Wire Wire Line
+	4250 6700 3700 6700
+Text Label 4250 6700 2    50   ~ 0
+BARO_FGND
+Wire Wire Line
+	4250 5900 3700 5900
+Text Label 4250 5900 2    50   ~ 0
+BARO_VDD
+Connection ~ 3700 5900
+Connection ~ 3700 6700
 $EndSCHEMATC

Commit message: Commit
Parts:
- gave numbers to parts that had none: 1
Changed lines of the file:
@@
 AR Path="/5ED663F7/5EE69A69" Ref="C?"  Part="1"
 AR Path="/5EF65A4D/5EF663FB/5EE69A69" Ref="C?"  Part="1"
-AR Path="/5EF65A4D/5EE69A69" Ref="C?"  Part="1"
+AR Path="/5EF65A4D/5EE69A69" Ref="C1"  Part="1"
 AR Path="/5EDADA57/5EE69A69" Ref="C?"  Part="1"
 AR Path="/5EF65A4D/5EE0D50D/5EE69A69" Ref="C?"  Part="1"
 AR Path="/5EE06F22/5EE2A025/5EE69A69" Ref="C?"  Part="1"
-F 0 "C?" H 3550 6400 50  0000 L CNN
+F 0 "C1" H 3550 6400 50  0000 L CNN
 F 1 "22uF/10V" H 3300 6200 50  0000 L CNN
 F 2 "Capacitor_SMD:C_1206_3216Metric" H 3738 6150 50  0001 C CNN
