File: HW/rbpi-z-hat/BQ24313.sch (KiCad schematic (older format))
At the start: 3 parts

Commit message: Commit...
Parts:
- R10, R9: renamed from R?; footprint (none) -> Resistor_SMD:R_0603_1608Metric
- gave numbers to parts that had none: 1
Connections:
- net labels added: BQ_IN, BQ_OUT, BQ_VSS, BQ_nCE, BQ_nFAULT
Changed lines of the file:
@@
 $Descr A4 8268 11693 portrait
 encoding utf-8
-Sheet 14 14
+Sheet 14 18
 Title "RasPi Zero NAV Hat"
 Date "2020-06-08"
@@
 P 3900 5450
 AR Path="/5EDDFB2B" Ref="IC?"  Part="1"
-AR Path="/5EDDEA36/5EDDFB2B" Ref="IC?"  Part="1"
-F 0 "IC?" H 4500 5715 50  0000 C CNN
+AR Path="/5EDDEA36/5EDDFB2B" Ref="IC1"  Part="1"
+F 0 "IC1" H 4500 5715 50  0000 C CNN
 F 1 "BQ24315DSGR" H 4500 5624 50  0000 C CNN
 F 2 "SON50P200X200X80-9N" H 4950 5550 50  0001 L CNN
@@
 $EndComp
 $Comp
-L power:GNDD #PWR?
+L power:GNDD #PWR0148
 U 1 1 5EDE0C1D
 P 4500 6450
-F 0 "#PWR?" H 4500 6200 50  0001 C CNN
+F 0 "#PWR0148" H 4500 6200 50  0001 C CNN
 F 1 "GNDD" H 4504 6295 50  0000 C CNN
 F 2 "" H 4500 6450 50  0001 C CNN
@@
 	5450 5650 5450 6350
 $Comp
-L power:GNDD #PWR?
+L power:GNDD #PWR0149
 U 1 1 5EDE184C
 P 5450 6350
-F 0 "#PWR?" H 5450 6100 50  0001 C CNN
+F 0 "#PWR0149" H 5450 6100 50  0001 C CNN
 F 1 "GNDD" H 5450 6200 50  0000 C CNN
 F 2 "" H 5450 6350 50  0001 C CNN
@@
 $EndComp
 $Comp
-L Device:R R?
+L Device:R R10
 U 1 1 5EDE259E
 P 5700 6050
-F 0 "R?" H 5770 6096 50  0000 L CNN
+F 0 "R10" H 5770 6096 50  0000 L CNN
 F 1 "25K" H 5770 6005 50  0000 L CNN
-F 2 "" V 5630 6050 50  0001 C CNN
+F 2 "Resistor_SMD:R_0603_1608Metric" V 5630 6050 50  0001 C CNN
 F 3 "~" H 5700 6050 50  0001 C CNN
 	1    5700 6050
@@
 	5700 6200 5700 6350
 $Comp
-L power:GNDD #PWR?
+L power:GNDD #PWR0150
 U 1 1 5EDE3539
 P 5700 6350
-F 0 "#PWR?" H 5700 6100 50  0001 C CNN
+F 0 "#PWR0150" H 5700 6100 50  0001 C CNN
 F 1 "GNDD" H 5750 6200 50  0000 C CNN
 F 2 "" H 5700 6350 50  0001 C CNN
@@
 $EndComp
 $Comp
-L Device:R R?
+L Device:R R9
 U 1 1 5EDE6B0A
 P 5150 6050
-F 0 "R?" H 5220 6096 50  0000 L CNN
+F 0 "R9" H 5220 6096 50  0000 L CNN
 F 1 "10K" H 5220 6005 50  0000 L CNN
-F 2 "" V 5080 6050 50  0001 C CNN
+F 2 "Resistor_SMD:R_0603_1608Metric" V 5080 6050 50  0001 C CNN
 F 3 "~" H 5150 6050 50  0001 C CNN
 	1    5150 6050
@@
 	5150 6200 5150 6350
 $Comp
-L power:GNDD #PWR?
+L power:GNDD #PWR0151
 U 1 1 5EDE6B11
 P 5150 6350
-F 0 "#PWR?" H 5150 6100 50  0001 C CNN
+F 0 "#PWR0151" H 5150 6100 50  0001 C CNN
 F 1 "GNDD" H 5150 6200 50  0000 C CNN
 F 2 "" H 5150 6350 50  0001 C CNN
@@
 	5100 5550 5700 5550
 Wire Wire Line
-	5150 5750 6000 5750
+	5150 5750 5900 5750
 Connection ~ 5150 5750
 Wire Wire Line
-	3900 5450 3400 5450
+	3900 5450 3600 5450
 Wire Wire Line
 	3900 5550 3800 5550
 Wire Wire Line
-	3900 5750 3400 5750
+	3900 5750 3600 5750
 Wire Wire Line
 	3800 5550 3800 6350
@@
 Connection ~ 3800 5550
 Wire Wire Line
-	3800 5550 3400 5550
+	3800 5550 3600 5550
 Connection ~ 4500 6350
 Wire Wire Line
 	4500 6350 4500 6450
 Wire Wire Line
-	5100 5450 6000 5450
+	5100 5450 5900 5450
+Text HLabel 3600 5450 0    50   Input ~ 0
+BQ_IN
+Text HLabel 3600 5550 0    50   Input ~ 0
+BQ_VSS
+Text HLabel 3600 5750 0    50   Output ~ 0
+BQ_nFAULT
+Text HLabel 5900 5450 2    50   Output ~ 0
+BQ_OUT
+Text HLabel 5900 5750 2    50   Output ~ 0
+BQ_nCE
 $EndSCHEMATC
