File: HW/rbpi-z-hat/I2C_CONN.sch (KiCad schematic (older format))
At the start: 9 parts

Commit message: Commit...
Parts:
- gave numbers to parts that had none: 9
Changed lines of the file:
@@
 $Descr A4 8268 11693 portrait
 encoding utf-8
-Sheet 10 14
+Sheet 9 18
 Title "RasPi Zero NAV Hat"
 Date "2020-06-08"
@@
 P 4750 3900
 AR Path="/5F0378CD/5EDD329B" Ref="C?"  Part="1"
-AR Path="/5EDD13AE/5EDD329B" Ref="C?"  Part="1"
-F 0 "C?" H 4750 4100 50  0000 C CNN
+AR Path="/5EDD13AE/5EDD329B" Ref="C5"  Part="1"
+F 0 "C5" H 4750 4100 50  0000 C CNN
 F 1 "1uF/16V/0805/NFM21PC105B1C3D" H 4750 4400 50  0000 C CNN
 F 2 "NFM21PC105B1C3D:NFM21PC105B1C3D" V 4750 3900 50  0001 C CNN
@@
 P 5200 4100
 AR Path="/5F0378CD/5EDD32A1" Ref="D?"  Part="1"
-AR Path="/5EDD13AE/5EDD32A1" Ref="D?"  Part="1"
-F 0 "D?" V 5050 4150 50  0000 L CNN
+AR Path="/5EDD13AE/5EDD32A1" Ref="D3"  Part="1"
+F 0 "D3" V 5050 4150 50  0000 L CNN
 F 1 "PESD0402-140" H 5200 4000 50  0000 C CNN
 F 2 "Diode_SMD:D_0402_1005Metric" H 5200 4100 50  0001 C CNN
@@
 P 4100 3800
 AR Path="/5F0378CD/5EDD32A7" Ref="FB?"  Part="1"
-AR Path="/5EDD13AE/5EDD32A7" Ref="FB?"  Part="1"
-F 0 "FB?" V 3826 3800 50  0000 C CNN
+AR Path="/5EDD13AE/5EDD32A7" Ref="FB3"  Part="1"
+F 0 "FB3" V 3826 3800 50  0000 C CNN
 F 1 "Ferrite_Bead" V 3917 3800 50  0000 C CNN
 F 2 "Inductor_SMD:L_0603_1608Metric" V 4030 3800 50  0001 C CNN
@@
 P 5200 4400
 AR Path="/5F0378CD/5EDD32B2" Ref="#PWR?"  Part="1"
-AR Path="/5EDD13AE/5EDD32B2" Ref="#PWR?"  Part="1"
-F 0 "#PWR?" H 5200 4150 50  0001 C CNN
+AR Path="/5EDD13AE/5EDD32B2" Ref="#PWR0107"  Part="1"
+F 0 "#PWR0107" H 5200 4150 50  0001 C CNN
 F 1 "GNDD" H 5204 4245 50  0000 C CNN
 F 2 "" H 5200 4400 50  0001 C CNN
@@
 P 4750 4100
 AR Path="/5F0378CD/5EDD32B8" Ref="#PWR?"  Part="1"
-AR Path="/5EDD13AE/5EDD32B8" Ref="#PWR?"  Part="1"
-F 0 "#PWR?" H 4750 3850 50  0001 C CNN
+AR Path="/5EDD13AE/5EDD32B8" Ref="#PWR0108"  Part="1"
+F 0 "#PWR0108" H 4750 3850 50  0001 C CNN
 F 1 "GNDD" H 4754 3945 50  0000 C CNN
 F 2 "" H 4750 4100 50  0001 C CNN
@@
 P 3700 3550
 AR Path="/5F0378CD/5EDD32C2" Ref="#PWR?"  Part="1"
-AR Path="/5EDD13AE/5EDD32C2" Ref="#PWR?"  Part="1"
-F 0 "#PWR?" H 3700 3400 50  0001 C CNN
+AR Path="/5EDD13AE/5EDD32C2" Ref="#PWR0109"  Part="1"
+F 0 "#PWR0109" H 3700 3400 50  0001 C CNN
 F 1 "+5V" H 3715 3723 50  0000 C CNN
 F 2 "" H 3700 3550 50  0001 C CNN
@@
 	4750 3650 4750 3450
 $Comp
-L Connector_Generic_MountingPin:Conn_01x04_MountingPin J?
+L Connector_Generic_MountingPin:Conn_01x04_MountingPin J9
 U 1 1 5EDD38F4
 P 6050 5700
-F 0 "J?" H 6050 5900 50  0000 C CNN
+F 0 "J9" H 6050 5900 50  0000 C CNN
 F 1 "JST_GH" V 6150 5700 50  0000 C CNN
 F 2 "Connector_JST:JST_GH_BM04B-GHS-TBT_1x04-1MP_P1.25mm_Vertical" H 6050 5700 50  0001 C CNN
@@
 $EndComp
 $Comp
-L power:GNDD #PWR?
+L power:GNDD #PWR0110
 U 1 1 5EDD6463
 P 5650 6600
-F 0 "#PWR?" H 5650 6350 50  0001 C CNN
+F 0 "#PWR0110" H 5650 6350 50  0001 C CNN
 F 1 "GNDD" H 5654 6445 50  0000 C CNN
 F 2 "" H 5650 6600 50  0001 C CNN
@@
 $EndComp
 $Comp
-L Device:Ferrite_Bead FB?
+L Device:Ferrite_Bead FB4
 U 1 1 5EDD6469
 P 5650 6250
-F 0 "FB?" H 5500 6200 50  0000 C CNN
+F 0 "FB4" H 5500 6200 50  0000 C CNN
 F 1 "Ferrite_Bead" H 5350 6400 50  0000 C CNN
 F 2 "Inductor_SMD:L_0603_1608Metric" V 5580 6250 50  0001 C CNN
@@
 	5650 6400 5650 6600
 $Comp
-L power:GNDD #PWR?
+L power:GNDD #PWR0111
 U 1 1 5EDD6470
 P 6050 6600
-F 0 "#PWR?" H 6050 6350 50  0001 C CNN
+F 0 "#PWR0111" H 6050 6350 50  0001 C CNN
 F 1 "GNDD" H 6054 6445 50  0000 C CNN
 F 2 "" H 6050 6600 50  0001 C CNN
@@
 	5650 5600 5850 5600
 $Comp
-L Interface:PCA9306DC U?
+L Interface:PCA9306DC U4
 U 1 1 5EDDAC68
 P 3750 5700
-F 0 "U?" H 3950 6150 50  0000 C CNN
+F 0 "U4" H 3950 6150 50  0000 C CNN
 F 1 "PCA9306DC" H 4000 5250 50  0000 C CNN
 F 2 "Package_SO:VSSOP-8_2.3x2mm_P0.5mm" H 3750 5250 50  0001 C CNN
@@
 $EndComp
 $Comp
-L power:GNDD #PWR?
+L power:GNDD #PWR0130
 U 1 1 5EDDD16D
 P 3750 6400
-F 0 "#PWR?" H 3750 6150 50  0001 C CNN
+F 0 "#PWR0130" H 3750 6150 50  0001 C CNN
 F 1 "GNDD" H 3754 6245 50  0000 C CNN
 F 2 "" H 3750 6400 50  0001 C CNN
@@
 	3750 6200 3750 6400
 $Comp
-L Power_Protection:SP0502BAHT D?
+L Power_Protection:SP0502BAHT D4
 U 1 1 5EDE2789
 P 5050 6250
-F 0 "D?" H 5200 6400 50  0000 L CNN
+F 0 "D4" H 5200 6400 50  0000 L CNN
 F 1 "PESD3V3S2UT" H 5050 6100 50  0000 L CNN
 F 2 "Package_TO_SOT_SMD:SOT-23" H 5275 6200 50  0001 L CNN
@@
 $EndComp
 $Comp
-L power:GNDD #PWR?
+L power:GNDD #PWR0131
 U 1 1 5EDE408B
 P 5050 6600
-F 0 "#PWR?" H 5050 6350 50  0001 C CNN
+F 0 "#PWR0131" H 5050 6350 50  0001 C CNN
 F 1 "GNDD" H 5054 6445 50  0000 C CNN
 F 2 "" H 5050 6600 50  0001 C CNN
@@
 	4950 6050 4950 5800
 $Comp
-L Device:R_Pack04 RN?
+L Device:R_Pack04 RN9
 U 1 1 5EDEDF2B
 P 3700 7100
-F 0 "RN?" V 3400 7100 50  0000 C CNN
+F 0 "RN9" V 3400 7100 50  0000 C CNN
 F 1 "1K5" V 3900 7100 50  0000 C CNN
 F 2 "Resistor_SMD:R_Array_Concave_4x0402" V 3975 7100 50  0001 C CNN
@@
 	5150 5700 5850 5700
 $Comp
-L power:+3.3V #PWR?
+L power:+3.3V #PWR0132
 U 1 1 5EE0BEF6
 P 3650 4700
-F 0 "#PWR?" H 3650 4550 50  0001 C CNN
+F 0 "#PWR0132" H 3650 4550 50  0001 C CNN
 F 1 "+3.3V" H 3800 4800 50  0000 C CNN
 F 2 "" H 3650 4700 50  0001 C CNN
@@
 $EndComp
 $Comp
-L Device:R R?
+L Device:R R1
 U 1 1 5EE0E2DE
 P 4100 4950
-F 0 "R?" H 4000 4950 50  0000 C CNN
+F 0 "R1" H 4000 4950 50  0000 C CNN
 F 1 "200K" V 4100 4950 50  0000 C CNN
 F 2 "Resistor_SMD:R_0603_1608Metric" V 4030 4950 50  0001 C CNN
@@
 Connection ~ 4100 5150
 $Comp
-L power:+3.3V #PWR?
+L power:+3.3V #PWR0133
 U 1 1 5EE2063C
 P 4100 4700
-F 0 "#PWR?" H 4100 4550 50  0001 C CNN
+F 0 "#PWR0133" H 4100 4550 50  0001 C CNN
 F 1 "+3.3V" H 4250 4800 50  0000 C CNN
 F 2 "" H 4100 4700 50  0001 C CNN
@@
 	4100 4700 4100 4800
 $Comp
-L power:+3.3V #PWR?
+L power:+3.3V #PWR0134
 U 1 1 5EE21A70
 P 3300 7350
-F 0 "#PWR?" H 3300 7200 50  0001 C CNN
+F 0 "#PWR0134" H 3300 7200 50  0001 C CNN
 F 1 "+3.3V" H 3300 7500 50  0000 C CNN
 F 2 "" H 3300 7350 50  0001 C CNN
