File: HW/rbpi-z-hat/MIC5504.sch (KiCad schematic (older format))
At the start: 3 parts

Commit message: Commit...
Parts:
- gave numbers to parts that had none: 3
Other:
- note added: "MIC5504-3.3YM5-TR\nor\nLP5907MFX-3.3"
- note removed: "MIC5504-3.3YM5-TR\nLP5907MFX-3.3"
Changed lines of the file:
@@
 $Descr A4 8268 11693 portrait
 encoding utf-8
-Sheet 13 14
+Sheet 12 18
 Title "RasPi Zero NAV Hat"
 Date "2020-06-08"
@@
 P 4400 5700
 AR Path="/5EDAE43F" Ref="U?"  Part="1"
-AR Path="/5EDADA57/5EDAE43F" Ref="U?"  Part="1"
-F 0 "U?" H 4400 6067 50  0000 C CNN
+AR Path="/5EDADA57/5EDAE43F" Ref="U7"  Part="1"
+AR Path="/5EF65A4D/5EE0D50D/5EDAE43F" Ref="U1"  Part="1"
+AR Path="/5EE06F22/5EE2A025/5EDAE43F" Ref="U11"  Part="1"
+F 0 "U11" H 4400 6067 50  0000 C CNN
 F 1 "MIC5504-3.3YM5" H 4400 5976 50  0000 C CNN
 F 2 "Package_TO_SOT_SMD:SOT-23-5" H 4400 5300 50  0001 C CNN
@@
 AR Path="/5EF65A4D/5EF663FB/5EDB342A" Ref="C?"  Part="1"
 AR Path="/5EF65A4D/5EDB342A" Ref="C?"  Part="1"
-AR Path="/5EDADA57/5EDB342A" Ref="C?"  Part="1"
-F 0 "C?" H 3250 6100 50  0000 L CNN
+AR Path="/5EDADA57/5EDB342A" Ref="C20"  Part="1"
+AR Path="/5EF65A4D/5EE0D50D/5EDB342A" Ref="C1"  Part="1"
+AR Path="/5EE06F22/5EE2A025/5EDB342A" Ref="C35"  Part="1"
+F 0 "C35" H 3250 6100 50  0000 L CNN
 F 1 "22uF/10V" H 3000 5900 50  0000 L CNN
 F 2 "Capacitor_SMD:C_1206_3216Metric" H 3438 5850 50  0001 C CNN
@@
 AR Path="/5EF65A4D/5EF663FB/5EDB5652" Ref="C?"  Part="1"
 AR Path="/5EF65A4D/5EDB5652" Ref="C?"  Part="1"
-AR Path="/5EDADA57/5EDB5652" Ref="C?"  Part="1"
-F 0 "C?" H 4950 6100 50  0000 L CNN
+AR Path="/5EDADA57/5EDB5652" Ref="C21"  Part="1"
+AR Path="/5EF65A4D/5EE0D50D/5EDB5652" Ref="C3"  Part="1"
+AR Path="/5EE06F22/5EE2A025/5EDB5652" Ref="C36"  Part="1"
+F 0 "C36" H 4950 6100 50  0000 L CNN
 F 1 "22uF/10V" H 4700 5900 50  0000 L CNN
 F 2 "Capacitor_SMD:C_1206_3216Metric" H 5138 5850 50  0001 C CNN
@@
 Connection ~ 4400 6400
 Text Notes 4000 5200 0    50   ~ 0
-MIC5504-3.3YM5-TR\nLP5907MFX-3.3
+MIC5504-3.3YM5-TR\nor\nLP5907MFX-3.3
 $EndSCHEMATC

Commit message: Commit
Changed lines of the file:
@@
 AR Path="/5EF65A4D/5EE0D50D/5EDAE43F" Ref="U1"  Part="1"
 AR Path="/5EE06F22/5EE2A025/5EDAE43F" Ref="U11"  Part="1"
-F 0 "U11" H 4400 6067 50  0000 C CNN
+F 0 "U7" H 4400 6067 50  0000 C CNN
 F 1 "MIC5504-3.3YM5" H 4400 5976 50  0000 C CNN
 F 2 "Package_TO_SOT_SMD:SOT-23-5" H 4400 5300 50  0001 C CNN
@@
 AR Path="/5EF65A4D/5EE0D50D/5EDB342A" Ref="C1"  Part="1"
 AR Path="/5EE06F22/5EE2A025/5EDB342A" Ref="C35"  Part="1"
-F 0 "C35" H 3250 6100 50  0000 L CNN
+F 0 "C20" H 3250 6100 50  0000 L CNN
 F 1 "22uF/10V" H 3000 5900 50  0000 L CNN
 F 2 "Capacitor_SMD:C_1206_3216Metric" H 3438 5850 50  0001 C CNN
@@
 AR Path="/5EF65A4D/5EE0D50D/5EDB5652" Ref="C3"  Part="1"
 AR Path="/5EE06F22/5EE2A025/5EDB5652" Ref="C36"  Part="1"
-F 0 "C36" H 4950 6100 50  0000 L CNN
+F 0 "C21" H 4950 6100 50  0000 L CNN
 F 1 "22uF/10V" H 4700 5900 50  0000 L CNN
 F 2 "Capacitor_SMD:C_1206_3216Metric" H 5138 5850 50  0001 C CNN

Commit message: Commit
Changed lines of the file:
@@
 AR Path="/5EF65A4D/5EE0D50D/5EDAE43F" Ref="U1"  Part="1"
 AR Path="/5EE06F22/5EE2A025/5EDAE43F" Ref="U11"  Part="1"
-AR Path="/5EE7A13E/5EE7A848/5EDAE43F" Ref="U?"  Part="1"
-F 0 "U7" H 4400 6067 50  0000 C CNN
+AR Path="/5EE7A13E/5EE7A848/5EDAE43F" Ref="U1"  Part="1"
+F 0 "U1" H 4400 6067 50  0000 C CNN
 F 1 "MIC5504-3.3YM5" H 4400 5976 50  0000 C CNN
 F 2 "Package_TO_SOT_SMD:SOT-23-5" H 4400 5300 50  0001 C CNN
@@
 AR Path="/5EF65A4D/5EE0D50D/5EDB342A" Ref="C1"  Part="1"
 AR Path="/5EE06F22/5EE2A025/5EDB342A" Ref="C35"  Part="1"
-AR Path="/5EE7A13E/5EE7A848/5EDB342A" Ref="C?"  Part="1"
-F 0 "C20" H 3250 6100 50  0000 L CNN
+AR Path="/5EE7A13E/5EE7A848/5EDB342A" Ref="C22"  Part="1"
+F 0 "C22" H 3250 6100 50  0000 L CNN
 F 1 "22uF/10V" H 3000 5900 50  0000 L CNN
 F 2 "Capacitor_SMD:C_1206_3216Metric" H 3438 5850 50  0001 C CNN
@@
 AR Path="/5EF65A4D/5EE0D50D/5EDB5652" Ref="C3"  Part="1"
 AR Path="/5EE06F22/5EE2A025/5EDB5652" Ref="C36"  Part="1"
-AR Path="/5EE7A13E/5EE7A848/5EDB5652" Ref="C?"  Part="1"
-F 0 "C21" H 4950 6100 50  0000 L CNN
+AR Path="/5EE7A13E/5EE7A848/5EDB5652" Ref="C31"  Part="1"
+F 0 "C31" H 4950 6100 50  0000 L CNN
 F 1 "22uF/10V" H 4700 5900 50  0000 L CNN
 F 2 "Capacitor_SMD:C_1206_3216Metric" H 5138 5850 50  0001 C CNN
