File: HW/rbpi-z-hat/POWER_CONN.sch (KiCad schematic (older format))
At the start: 13 parts

Commit message: Commit...
Parts:
- C18, C19: renamed from C?; value 1uF/16V/0805/NFM21PC105B1C3D -> 1uF/16V/NFM21PC105B1C3D
- gave numbers to parts that had none: 11
Changed lines of the file:
@@
 $Descr A4 8268 11693 portrait
 encoding utf-8
-Sheet 12 14
+Sheet 12 18
 Title "RasPi Zero NAV Hat"
 Date "2020-06-08"
@@
 $EndDescr
 $Comp
-L Connector_Generic_MountingPin:Conn_01x06_MountingPin J?
+L Connector_Generic_MountingPin:Conn_01x06_MountingPin J10
 U 1 1 5EF28CAE
 P 2750 3700
-F 0 "J?" H 2750 4000 50  0000 C CNN
+F 0 "J10" H 2750 4000 50  0000 C CNN
 F 1 "JST_GH" V 2850 3650 50  0000 C CNN
 F 2 "Connector_JST:JST_GH_BM06B-GHS-TBT_1x06-1MP_P1.25mm_Vertical" H 2750 3700 50  0001 C CNN
@@
 P 3050 4700
 AR Path="/5F0378CD/5EDAAF84" Ref="#PWR?"  Part="1"
-AR Path="/5EF28018/5EDAAF84" Ref="#PWR?"  Part="1"
-F 0 "#PWR?" H 3050 4450 50  0001 C CNN
+AR Path="/5EF28018/5EDAAF84" Ref="#PWR0138"  Part="1"
+F 0 "#PWR0138" H 3050 4450 50  0001 C CNN
 F 1 "GNDD" H 3054 4545 50  0000 C CNN
 F 2 "" H 3050 4700 50  0001 C CNN
@@
 P 3050 4350
 AR Path="/5F0378CD/5EDAAF8A" Ref="FB?"  Part="1"
-AR Path="/5EF28018/5EDAAF8A" Ref="FB?"  Part="1"
-F 0 "FB?" H 2950 4250 50  0000 C CNN
+AR Path="/5EF28018/5EDAAF8A" Ref="FB6"  Part="1"
+F 0 "FB6" H 2950 4250 50  0000 C CNN
 F 1 "MPZ2012S221AT000" V 3200 4400 50  0000 C CNN
 F 2 "Inductor_SMD:L_0805_2012Metric" V 2980 4350 50  0001 C CNN
@@
 P 2750 4700
 AR Path="/5F0378CD/5EDAAF91" Ref="#PWR?"  Part="1"
-AR Path="/5EF28018/5EDAAF91" Ref="#PWR?"  Part="1"
-F 0 "#PWR?" H 2750 4450 50  0001 C CNN
+AR Path="/5EF28018/5EDAAF91" Ref="#PWR0139"  Part="1"
+F 0 "#PWR0139" H 2750 4450 50  0001 C CNN
 F 1 "GNDD" H 2754 4545 50  0000 C CNN
 F 2 "" H 2750 4700 50  0001 C CNN
@@
 AR Path="/5EF65A4D/5EDAD60C" Ref="C?"  Part="1"
 AR Path="/5EF0850C/5EDAD60C" Ref="C?"  Part="1"
-AR Path="/5EF28018/5EDAD60C" Ref="C?"  Part="1"
-F 0 "C?" H 4050 4200 50  0000 L CNN
+AR Path="/5EF28018/5EDAD60C" Ref="C11"  Part="1"
+F 0 "C11" H 4050 4200 50  0000 L CNN
 F 1 "22uF/16V" H 3800 4000 50  0000 L CNN
 F 2 "Capacitor_SMD:C_1210_3225Metric" H 4238 3950 50  0001 C CNN
@@
 AR Path="/5F0378CD/5EDB1BFC" Ref="D?"  Part="1"
 AR Path="/5EDD13AE/5EDB1BFC" Ref="D?"  Part="1"
-AR Path="/5EF28018/5EDB1BFC" Ref="D?"  Part="1"
-F 0 "D?" V 3650 4150 50  0000 L CNN
+AR Path="/5EF28018/5EDB1BFC" Ref="D5"  Part="1"
+F 0 "D5" V 3650 4150 50  0000 L CNN
 F 1 "PESD0402-140" H 3800 4000 50  0000 C CNN
 F 2 "Diode_SMD:D_0402_1005Metric" H 3800 4100 50  0001 C CNN
@@
 AR Path="/5F0378CD/5EDB1C02" Ref="FB?"  Part="1"
 AR Path="/5EDD13AE/5EDB1C02" Ref="FB?"  Part="1"
-AR Path="/5EF28018/5EDB1C02" Ref="FB?"  Part="1"
-F 0 "FB?" V 4226 3500 50  0000 C CNN
+AR Path="/5EF28018/5EDB1C02" Ref="FB5"  Part="1"
+F 0 "FB5" V 4226 3500 50  0000 C CNN
 F 1 "MPZ2012S221AT000" V 4317 3500 50  0000 C CNN
 F 2 "Inductor_SMD:L_0805_2012Metric" V 4430 3500 50  0001 C CNN
@@
 AR Path="/5F0378CD/5EDB1C0D" Ref="#PWR?"  Part="1"
 AR Path="/5EDD13AE/5EDB1C0D" Ref="#PWR?"  Part="1"
-AR Path="/5EF28018/5EDB1C0D" Ref="#PWR?"  Part="1"
-F 0 "#PWR?" H 3800 4450 50  0001 C CNN
+AR Path="/5EF28018/5EDB1C0D" Ref="#PWR0140"  Part="1"
+F 0 "#PWR0140" H 3800 4450 50  0001 C CNN
 F 1 "GNDD" H 3804 4545 50  0000 C CNN
 F 2 "" H 3800 4700 50  0001 C CNN
@@
 AR Path="/5F0378CD/5EDB27EB" Ref="C?"  Part="1"
 AR Path="/5EDD13AE/5EDB27EB" Ref="C?"  Part="1"
-AR Path="/5EF28018/5EDB27EB" Ref="C?"  Part="1"
-F 0 "C?" H 3200 6700 50  0000 C CNN
-F 1 "1uF/16V/0805/NFM21PC105B1C3D" H 3200 6800 50  0000 C CNN
+AR Path="/5EF28018/5EDB27EB" Ref="C18"  Part="1"
+F 0 "C18" H 3200 6700 50  0000 C CNN
+F 1 "1uF/16V/NFM21PC105B1C3D" H 3200 6800 50  0000 C CNN
 F 2 "NFM21PC105B1C3D:NFM21PC105B1C3D" V 3200 6500 50  0001 C CNN
 F 3 "~" V 3200 6500 50  0001 C CNN
@@
 AR Path="/5F0378CD/5EDB7712" Ref="#PWR?"  Part="1"
 AR Path="/5EDD13AE/5EDB7712" Ref="#PWR?"  Part="1"
-AR Path="/5EF28018/5EDB7712" Ref="#PWR?"  Part="1"
-F 0 "#PWR?" H 4200 4450 50  0001 C CNN
+AR Path="/5EF28018/5EDB7712" Ref="#PWR0141"  Part="1"
+F 0 "#PWR0141" H 4200 4450 50  0001 C CNN
 F 1 "GNDD" H 4204 4545 50  0000 C CNN
 F 2 "" H 4200 4700 50  0001 C CNN
@@
 AR Path="/5F0378CD/5EDBBE20" Ref="#PWR?"  Part="1"
 AR Path="/5EDD13AE/5EDBBE20" Ref="#PWR?"  Part="1"
-AR Path="/5EF28018/5EDBBE20" Ref="#PWR?"  Part="1"
-F 0 "#PWR?" H 3200 6800 50  0001 C CNN
+AR Path="/5EF28018/5EDBBE20" Ref="#PWR0142"  Part="1"
+F 0 "#PWR0142" H 3200 6800 50  0001 C CNN
 F 1 "GNDD" H 3204 6895 50  0000 C CNN
 F 2 "" H 3200 7050 50  0001 C CNN
@@
 $EndComp
 $Comp
-L Device:R R?
+L Device:R R3
 U 1 1 5EDBC79D
 P 2900 6750
-F 0 "R?" H 2970 6796 50  0000 L CNN
+F 0 "R3" H 2970 6796 50  0000 L CNN
 F 1 "1M" H 2970 6705 50  0000 L CNN
 F 2 "Inductor_SMD:L_0603_1608Metric" V 2830 6750 50  0001 C CNN
@@
 AR Path="/5F0378CD/5EDBD7B6" Ref="#PWR?"  Part="1"
 AR Path="/5EDD13AE/5EDBD7B6" Ref="#PWR?"  Part="1"
-AR Path="/5EF28018/5EDBD7B6" Ref="#PWR?"  Part="1"
-F 0 "#PWR?" H 2900 6800 50  0001 C CNN
+AR Path="/5EF28018/5EDBD7B6" Ref="#PWR0143"  Part="1"
+F 0 "#PWR0143" H 2900 6800 50  0001 C CNN
 F 1 "GNDD" H 2904 6895 50  0000 C CNN
 F 2 "" H 2900 7050 50  0001 C CNN
@@
 $EndComp
 $Comp
-L Device:R_Pack04 RN?
+L Device:R_Pack04 RN10
 U 1 1 5EDA51BA
 P 4450 6600
-F 0 "RN?" V 4033 6600 50  0000 C CNN
+F 0 "RN10" V 4033 6600 50  0000 C CNN
 F 1 "10K/1%" V 4124 6600 50  0000 C CNN
 F 2 "Resistor_SMD:R_Array_Concave_4x0402" V 4725 6600 50  0001 C CNN
@@
 AR Path="/5F0378CD/5EDA9893" Ref="#PWR?"  Part="1"
 AR Path="/5EDD13AE/5EDA9893" Ref="#PWR?"  Part="1"
-AR Path="/5EF28018/5EDA9893" Ref="#PWR?"  Part="1"
-F 0 "#PWR?" H 4150 6550 50  0001 C CNN
+AR Path="/5EF28018/5EDA9893" Ref="#PWR0144"  Part="1"
+F 0 "#PWR0144" H 4150 6550 50  0001 C CNN
 F 1 "GNDD" H 4154 6645 50  0000 C CNN
 F 2 "" H 4150 6800 50  0001 C CNN
@@
 AR Path="/5F0378CD/5EDAC9C3" Ref="C?"  Part="1"
 AR Path="/5EDD13AE/5EDAC9C3" Ref="C?"  Part="1"
-AR Path="/5EF28018/5EDAC9C3" Ref="C?"  Part="1"
-F 0 "C?" H 3200 7850 50  0000 C CNN
-F 1 "1uF/16V/0805/NFM21PC105B1C3D" H 3200 7950 50  0000 C CNN
+AR Path="/5EF28018/5EDAC9C3" Ref="C19"  Part="1"
+F 0 "C19" H 3200 7850 50  0000 C CNN
+F 1 "1uF/16V/NFM21PC105B1C3D" H 3200 7950 50  0000 C CNN
 F 2 "NFM21PC105B1C3D:NFM21PC105B1C3D" V 3200 7650 50  0001 C CNN
 F 3 "~" V 3200 7650 50  0001 C CNN
@@
 AR Path="/5F0378CD/5EDAC9CC" Ref="#PWR?"  Part="1"
 AR Path="/5EDD13AE/5EDAC9CC" Ref="#PWR?"  Part="1"
-AR Path="/5EF28018/5EDAC9CC" Ref="#PWR?"  Part="1"
-F 0 "#PWR?" H 3200 7950 50  0001 C CNN
+AR Path="/5EF28018/5EDAC9CC" Ref="#PWR0145"  Part="1"
+F 0 "#PWR0145" H 3200 7950 50  0001 C CNN
 F 1 "GNDD" H 3204 8045 50  0000 C CNN
 F 2 "" H 3200 8200 50  0001 C CNN
@@
 $EndComp
 $Comp
-L Device:R R?
+L Device:R R8
 U 1 1 5EDAC9D2
 P 2900 7900
-F 0 "R?" H 2970 7946 50  0000 L CNN
+F 0 "R8" H 2970 7946 50  0000 L CNN
 F 1 "1M" H 2970 7855 50  0000 L CNN
 F 2 "Inductor_SMD:L_0603_1608Metric" V 2830 7900 50  0001 C CNN
@@
 AR Path="/5F0378CD/5EDAC9DC" Ref="#PWR?"  Part="1"
 AR Path="/5EDD13AE/5EDAC9DC" Ref="#PWR?"  Part="1"
-AR Path="/5EF28018/5EDAC9DC" Ref="#PWR?"  Part="1"
-F 0 "#PWR?" H 2900 7950 50  0001 C CNN
+AR Path="/5EF28018/5EDAC9DC" Ref="#PWR0146"  Part="1"
+F 0 "#PWR0146" H 2900 7950 50  0001 C CNN
 F 1 "GNDD" H 2904 8045 50  0000 C CNN
 F 2 "" H 2900 8200 50  0001 C CNN
@@
 	4000 6500 4250 6500
 $Comp
-L Device:R R?
+L Device:R R2
 U 1 1 5EDB2F43
 P 3650 6400
-F 0 "R?" V 3750 6400 50  0000 C CNN
+F 0 "R2" V 3750 6400 50  0000 C CNN
 F 1 "10K/0.1%" V 3550 6400 50  0000 C CNN
 F 2 "Inductor_SMD:L_0603_1608Metric" V 3580 6400 50  0001 C CNN
@@
 	3800 6400 4250 6400
 $Comp
-L Device:R R?
+L Device:R R7
 U 1 1 5EDB584F
 P 3650 7550
-F 0 "R?" V 3750 7550 50  0000 C CNN
+F 0 "R7" V 3750 7550 50  0000 C CNN
 F 1 "10K/0.1%" V 3550 7550 50  0000 C CNN
 F 2 "Inductor_SMD:L_0603_1608Metric" V 3580 7550 50  0001 C CNN
@@
 AR Path="/5EF65A4D/5EDC6AFF" Ref="C?"  Part="1"
 AR Path="/5EF0850C/5EDC6AFF" Ref="C?"  Part="1"
-AR Path="/5EF28018/5EDC6AFF" Ref="C?"  Part="1"
-F 0 "C?" H 4700 4200 50  0000 L CNN
+AR Path="/5EF28018/5EDC6AFF" Ref="C17"  Part="1"
+F 0 "C17" H 4700 4200 50  0000 L CNN
 F 1 "22uF/16V" H 4450 4000 50  0000 L CNN
 F 2 "Capacitor_SMD:C_1210_3225Metric" H 4888 3950 50  0001 C CNN
@@
 AR Path="/5F0378CD/5EDC6B06" Ref="#PWR?"  Part="1"
 AR Path="/5EDD13AE/5EDC6B06" Ref="#PWR?"  Part="1"
-AR Path="/5EF28018/5EDC6B06" Ref="#PWR?"  Part="1"
-F 0 "#PWR?" H 4850 4450 50  0001 C CNN
+AR Path="/5EF28018/5EDC6B06" Ref="#PWR0147"  Part="1"
+F 0 "#PWR0147" H 4850 4450 50  0001 C CNN
 F 1 "GNDD" H 4854 4545 50  0000 C CNN
 F 2 "" H 4850 4700 50  0001 C CNN
