File: HW/rbpi-z-hat/SENSORS_POWER.sch (KiCad schematic (older format))
At the start: 3 parts

Commit message: Commit
Parts:
- gave numbers to parts that had none: 3
Changed lines of the file:
@@
 AR Path="/5EF65A4D/5EE7A82C" Ref="L?"  Part="1"
 AR Path="/5EE06F22/5EE7A82C" Ref="L?"  Part="1"
-AR Path="/5EE7A13E/5EE7A82C" Ref="L?"  Part="1"
-F 0 "L?" V 4450 5250 50  0000 C CNN
+AR Path="/5EE7A13E/5EE7A82C" Ref="L2"  Part="1"
+F 0 "L2" V 4450 5250 50  0000 C CNN
 F 1 "Ferrite_Bead" V 4350 5250 50  0000 C CNN
 F 2 "Inductor_SMD:L_0603_1608Metric" V 4130 5250 50  0001 C CNN
@@
 AR Path="/5EF65A4D/5EE7A832" Ref="C?"  Part="1"
 AR Path="/5EE06F22/5EE7A832" Ref="C?"  Part="1"
-AR Path="/5EE7A13E/5EE7A832" Ref="C?"  Part="1"
-F 0 "C?" H 3900 5900 50  0000 L CNN
+AR Path="/5EE7A13E/5EE7A832" Ref="C12"  Part="1"
+F 0 "C12" H 3900 5900 50  0000 L CNN
 F 1 "100nF" H 3900 5700 50  0000 L CNN
 F 2 "Capacitor_SMD:C_0603_1608Metric" H 3888 5650 50  0001 C CNN
@@
 AR Path="/5EF65A4D/5EE7A83D" Ref="L?"  Part="1"
 AR Path="/5EE06F22/5EE7A83D" Ref="L?"  Part="1"
-AR Path="/5EE7A13E/5EE7A83D" Ref="L?"  Part="1"
-F 0 "L?" V 4400 6350 50  0000 C CNN
+AR Path="/5EE7A13E/5EE7A83D" Ref="L3"  Part="1"
+F 0 "L3" V 4400 6350 50  0000 C CNN
 F 1 "Ferrite_Bead" V 4050 6350 50  0000 C CNN
 F 2 "Inductor_SMD:L_0603_1608Metric" V 4130 6350 50  0001 C CNN

Commit message: Changes in Sch
Connections:
- net sheet5EE7A825/MIC_VIN renamed MIC5504/MIC_VIN
Changed lines of the file:
@@
 $Descr A4 8268 11693 portrait
 encoding utf-8
-Sheet 16 18
+Sheet 15 17
 Title "RasPi Zero NAV Hat"
 Date "2020-08-11"
@@
 S 4850 5150 900  400
 U 5EE7A848
-F0 "sheet5EE7A825" 50
+F0 "MIC5504" 50
 F1 "MIC5504.sch" 50
 F2 "MIC_EN" I L 4850 5350 50
