File: HW/rbpi-z-hat/PCA9685.sch (KiCad schematic (older format))
At the start: 19 parts, among them J2 Conn_01x10, J3 Conn_01x10, J4 Conn_01x10, J5 Conn_01x06, J6 Conn_01x06, J7 Conn_01x06, U3 PCA9685BS, X1 ASEMB-25.000MHZ-LC-T

Commit message: Updated PCA9685.sch
Connections:
- net SERVO_POWER: now reaches J3.1 (Pin_1), J3.10 (Pin_10), J3.2 (Pin_2), J3.3 (Pin_3), J3.4 (Pin_4), J3.5 (Pin_5), J3.6 (Pin_6), J3.7 (Pin_7), J3.8 (Pin_8), J3.9 (Pin_9), J6.1 (Pin_1), J6.2 (Pin_2), J6.3 (Pin_3), J6.4 (Pin_4), J6.5 (Pin_5), J6.6 (Pin_6)
Changed lines of the file:
@@
 	7150 8850 7150 9150
 Connection ~ 7150 9150
+Text HLabel 6500 7650 0    50   Input ~ 0
+SERVO_POWER
+Wire Wire Line
+	6550 7650 6500 7650
 $EndSCHEMATC
