File: HW/rbpi-z-hat/IST8310.kicad_sch (KiCad schematic)
At the start: 6 parts, among them U3 IST8310

Commit message: Added schematics for QMC5883L
Parts:
- added JP1, JP3: SolderJumper_3_Open, Jumper:SolderJumper-3_P1.3mm_Open_RoundedPad1.0x1.5mm_NumberLabels, symbol Jumper:SolderJumper_3_Open
Connections:
- net IST_GND: now also JP1.3 (B), JP3.3 (B)
- net IST_VDD: now also JP1.1 (A), JP3.1 (A)
- net at U3.5 (CAD0): now also JP3.2 (C)
- net at U3.6 (CAD1): now also JP1.2 (C)
Changed lines of the file:
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@@
     (comment 2 "Denis Tsekh")
   )
+  (junction (at 142.24 148.59) (diameter 0) (color 0 0 0 0)
+  )
   (junction (at 115.57 115.57) (diameter 0) (color 0 0 0 0)
   )
   (junction (at 128.27 125.73) (diameter 0) (color 0 0 0 0)
   )
+  (junction (at 113.03 158.75) (diameter 0) (color 0 0 0 0)
+  )
   (junction (at 113.03 115.57) (diameter 0) (color 0 0 0 0)
   )
@@
   (junction (at 91.44 115.57) (diameter 0) (color 0 0 0 0)
   )
+  (junction (at 132.08 115.57) (diameter 0) (color 0 0 0 0)
+  )
+  (junction (at 142.24 177.8) (diameter 0) (color 0 0 0 0)
+  )
   (junction (at 97.79 142.24) (diameter 0) (color 0 0 0 0)
   )
@@
     (stroke (width 0) (type default))
   )
+  (wire (pts (xy 124.46 168.91) (xy 144.78 168.91))
+    (stroke (width 0) (type default))
+  )
   (wire (pts (xy 132.08 124.46) (xy 132.08 125.73))
     (stroke (width 0) (type default))
@@
     (stroke (width 0) (type default))
   )
+  (wire (pts (xy 148.59 163.83) (xy 148.59 148.59))
+    (stroke (width 0) (type default))
+  )
+  (wire (pts (xy 142.24 148.59) (xy 142.24 153.67))
+    (stroke (width 0) (type default))
+  )
   (wire (pts (xy 97.79 115.57) (xy 97.79 130.81))
     (stroke (width 0) (type default))
@@
     (stroke (width 0) (type default))
   )
+  (wire (pts (xy 123.19 147.32) (xy 127 147.32))
+    (stroke (width 0) (type default))
+  )
   (wire (pts (xy 124.46 124.46) (xy 124.46 125.73))
     (stroke (width 0) (type default))
@@
     (stroke (width 0) (type default))
   )
+  (wire (pts (xy 132.08 115.57) (xy 142.24 115.57))
+    (stroke (width 0) (type default))
+  )
+  (wire (pts (xy 142.24 163.83) (xy 142.24 177.8))
+    (stroke (width 0) (type default))
+  )
+  (wire (pts (xy 148.59 177.8) (xy 148.59 173.99))
+    (stroke (width 0) (type default))
+  )
+  (wire (pts (xy 113.03 177.8) (xy 142.24 177.8))
+    (stroke (width 0) (type default))
+  )
   (wire (pts (xy 96.52 158.75) (xy 113.03 158.75))
     (stroke (width 0) (type default))
@@
     (stroke (width 0) (type default))
   )
+  (wire (pts (xy 124.46 149.86) (xy 124.46 168.91))
+    (stroke (width 0) (type default))
+  )
   (wire (pts (xy 129.54 134.62) (xy 129.54 135.89))
     (stroke (width 0) (type default))
   )
+  (wire (pts (xy 142.24 115.57) (xy 142.24 148.59))
+    (stroke (width 0) (type default))
+  )
+  (wire (pts (xy 127 158.75) (xy 138.43 158.75))
+    (stroke (width 0) (type default))
+  )
   (wire (pts (xy 128.27 128.27) (xy 137.16 128.27))
     (stroke (width 0) (type default))
@@
     (stroke (width 0) (type default))
   )
+  (wire (pts (xy 113.03 158.75) (xy 113.03 177.8))
+    (stroke (width 0) (type default))
+  )
   (wire (pts (xy 113.03 115.57) (xy 113.03 129.54))
     (stroke (width 0) (type default))
@@
     (stroke (width 0) (type default))
   )
+  (wire (pts (xy 148.59 148.59) (xy 142.24 148.59))
+    (stroke (width 0) (type default))
+  )
   (wire (pts (xy 123.19 139.7) (xy 125.73 139.7))
     (stroke (width 0) (type default))
   )
+  (wire (pts (xy 142.24 177.8) (xy 148.59 177.8))
+    (stroke (width 0) (type default))
+  )
   (wire (pts (xy 113.03 115.57) (xy 115.57 115.57))
     (stroke (width 0) (type default))
   )
+  (wire (pts (xy 123.19 149.86) (xy 124.46 149.86))
+    (stroke (width 0) (type default))
+  )
   (wire (pts (xy 91.44 139.7) (xy 102.87 139.7))
     (stroke (width 0) (type default))
@@
   )
   (wire (pts (xy 129.54 143.51) (xy 129.54 146.05))
+    (stroke (width 0) (type default))
+  )
+  (wire (pts (xy 127 147.32) (xy 127 158.75))
     (stroke (width 0) (type default))
   )
@@
   (hierarchical_label "IST_SCL" (shape input) (at 82.55 142.24 180) (fields_autoplaced)
     (effects (font (size 1.27 1.27)) (justify right))
+  )
+  (symbol (lib_id "Jumper:SolderJumper_3_Open") (at 142.24 158.75 270) (unit 1)
+    (in_bom yes) (on_board yes) (dnp no) (fields_autoplaced)
+    (property "Reference" "JP3" (at 144.78 157.48 90)
+      (effects (font (size 1.27 1.27)) (justify left))
+    )
+    (property "Value" "SolderJumper_3_Open" (at 144.78 160.02 90)
+      (effects (font (size 1.27 1.27)) (justify left))
+    )
+    (property "Footprint" "Jumper:SolderJumper-3_P1.3mm_Open_RoundedPad1.0x1.5mm_NumberLabels" (at 142.24 158.75 0)
+      (effects (font (size 1.27 1.27)) hide)
+    )
+    (property "Datasheet" "~" (at 142.24 158.75 0)
+      (effects (font (size 1.27 1.27)) hide)
+    )
+    (pin "1")
+    (pin "3")
+    (pin "2")
+    (instances
+      (project "rbpi-z-hat"
+        (path "/d99b0340-d795-4b40-9cde-9851c6cee99d/740a9ed9-3c23-4e4f-8dd1-04f07ce4215e/6911857f-8b28-442d-83af-e9e9a964ef3c"
+          (reference "JP3") (unit 1)
+        )
+      )
+    )
   )
   (symbol (lib_id "Device:C") (at 124.46 120.65 0) (unit 1)
@@
         )
       )
+    )
+  )
+  (symbol (lib_id "Jumper:SolderJumper_3_Open") (at 148.59 168.91 270) (unit 1)
+    (in_bom yes) (on_board yes) (dnp no) (fields_autoplaced)
+    (property "Reference" "JP1" (at 151.13 167.64 90)
+      (effects (font (size 1.27 1.27)) (justify left))
+    )
+    (property "Value" "SolderJumper_3_Open" (at 151.13 170.18 90)
+      (effects (font (size 1.27 1.27)) (justify left))
+    )
+    (property "Footprint" "Jumper:SolderJumper-3_P1.3mm_Open_RoundedPad1.0x1.5mm_NumberLabels" (at 148.59 168.91 0)
+      (effects (font (size 1.27 1.27)) hide)
+    )
+    (property "Datasheet" "~" (at 148.59 168.91 0)
+      (effects (font (size 1.27 1.27)) hide)
+    )
+    (pin "1")
+    (pin "3")
+    (pin "2")
+    (instances
+      (project "rbpi-z-hat"
+        (path "/d99b0340-d795-4b40-9cde-9851c6cee99d/740a9ed9-3c23-4e4f-8dd1-04f07ce4215e/6911857f-8b28-442d-83af-e9e9a964ef3c"
+          (reference "JP1") (unit 1)
+        )
+      )

Commit message: Apdated Sch and PCB
Parts:
- removed R4, R5: 4K7, Resistor_SMD:R_0402_1005Metric, symbol Device:R
Changed lines of the file:
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@@
   (junction (at 113.03 115.57) (diameter 0) (color 0 0 0 0)
   )
-  (junction (at 97.79 115.57) (diameter 0) (color 0 0 0 0)
-  )
-  (junction (at 91.44 115.57) (diameter 0) (color 0 0 0 0)
-  )
   (junction (at 132.08 115.57) (diameter 0) (color 0 0 0 0)
   )
   (junction (at 142.24 177.8) (diameter 0) (color 0 0 0 0)
   )
-  (junction (at 97.79 142.24) (diameter 0) (color 0 0 0 0)
-  )
   (junction (at 110.49 115.57) (diameter 0) (color 0 0 0 0)
   )
   (junction (at 124.46 115.57) (diameter 0) (color 0 0 0 0)
   )
-  (junction (at 91.44 139.7) (diameter 0) (color 0 0 0 0)
-  )
-  (wire (pts (xy 91.44 115.57) (xy 97.79 115.57))
+  (wire (pts (xy 82.55 115.57) (xy 110.49 115.57))
     (stroke (width 0) (type default))
   )
@@
     (stroke (width 0) (type default))
   )
-  (wire (pts (xy 97.79 115.57) (xy 97.79 130.81))
-    (stroke (width 0) (type default))
-  )
   (wire (pts (xy 129.54 146.05) (xy 138.43 146.05))
     (stroke (width 0) (type default))
@@
     (stroke (width 0) (type default))
   )
-  (wire (pts (xy 82.55 115.57) (xy 91.44 115.57))
-    (stroke (width 0) (type default))
-  )
   (wire (pts (xy 82.55 144.78) (xy 102.87 144.78))
     (stroke (width 0) (type default))
   )
-  (wire (pts (xy 91.44 138.43) (xy 91.44 139.7))
-    (stroke (width 0) (type default))
-  )
   (wire (pts (xy 132.08 116.84) (xy 132.08 115.57))
     (stroke (width 0) (type default))
@@
     (stroke (width 0) (type default))
   )
-  (wire (pts (xy 97.79 142.24) (xy 102.87 142.24))
+  (wire (pts (xy 82.55 142.24) (xy 102.87 142.24))
     (stroke (width 0) (type default))
   )
@@
     (stroke (width 0) (type default))
   )
-  (wire (pts (xy 82.55 142.24) (xy 97.79 142.24))
-    (stroke (width 0) (type default))
-  )
-  (wire (pts (xy 82.55 139.7) (xy 91.44 139.7))
+  (wire (pts (xy 82.55 139.7) (xy 102.87 139.7))
     (stroke (width 0) (type default))
   )
@@
     (stroke (width 0) (type default))
   )
-  (wire (pts (xy 97.79 115.57) (xy 110.49 115.57))
-    (stroke (width 0) (type default))
-  )
   (wire (pts (xy 110.49 115.57) (xy 110.49 129.54))
     (stroke (width 0) (type default))
@@
     (stroke (width 0) (type default))
   )
-  (wire (pts (xy 91.44 139.7) (xy 102.87 139.7))
-    (stroke (width 0) (type default))
-  )
   (wire (pts (xy 113.03 158.75) (xy 113.03 154.94))
     (stroke (width 0) (type default))
@@
   )
   (wire (pts (xy 127 147.32) (xy 127 158.75))
-    (stroke (width 0) (type default))
-  )
-  (wire (pts (xy 91.44 115.57) (xy 91.44 130.81))
-    (stroke (width 0) (type default))
-  )
-  (wire (pts (xy 97.79 138.43) (xy 97.79 142.24))
     (stroke (width 0) (type default))
   )
@@
         (path "/d99b0340-d795-4b40-9cde-9851c6cee99d/740a9ed9-3c23-4e4f-8dd1-04f07ce4215e/6911857f-8b28-442d-83af-e9e9a964ef3c"
           (reference "C6") (unit 1)
-        )
-      )
-    )
-  )
-  (symbol (lib_id "Device:R") (at 97.79 134.62 0) (unit 1)
-    (in_bom yes) (on_board yes) (dnp no)
-    (property "Reference" "R4" (at 99.06 133.35 0)
-      (effects (font (size 1.27 1.27)) (justify left))
-    )
-    (property "Value" "4K7" (at 99.06 135.89 0)
-      (effects (font (size 1.27 1.27)) (justify left))
-    )
-    (property "Footprint" "Resistor_SMD:R_0402_1005Metric" (at 96.012 134.62 90)
-      (effects (font (size 1.27 1.27)) hide)
-    )
-    (property "Datasheet" "~" (at 97.79 134.62 0)
-      (effects (font (size 1.27 1.27)) hide)
-    )
-    (pin "1")
-    (pin "2")
-    (instances
-      (project "rbpi-z-hat"
-        (path "/d99b0340-d795-4b40-9cde-9851c6cee99d/740a9ed9-3c23-4e4f-8dd1-04f07ce4215e/6911857f-8b28-442d-83af-e9e9a964ef3c"
-          (reference "R4") (unit 1)
         )
       )
@@
         )
       )
-    )
-  )
-  (symbol (lib_id "Device:R") (at 91.44 134.62 0) (unit 1)
-    (in_bom yes) (on_board yes) (dnp no)
-    (property "Reference" "R5" (at 92.71 133.35 0)
-      (effects (font (size 1.27 1.27)) (justify left))
-    )
-    (property "Value" "4K7" (at 92.71 135.89 0)
-      (effects (font (size 1.27 1.27)) (justify left))
-    )
-    (property "Footprint" "Resistor_SMD:R_0402_1005Metric" (at 89.662 134.62 90)
-      (effects (font (size 1.27 1.27)) hide)
-    )
-    (property "Datasheet" "~" (at 91.44 134.62 0)
-      (effects (font (size 1.27 1.27)) hide)
-    )
-    (pin "1")
-    (pin "2")
-    (instances
-      (project "rbpi-z-hat"
-        (path "/d99b0340-d795-4b40-9cde-9851c6cee99d/740a9ed9-3c23-4e4f-8dd1-04f07ce4215e/6911857f-8b28-442d-83af-e9e9a964ef3c"
-          (reference "R5") (unit 1)
-        )
-      )
