File: HW/rbpi-z-hat/BMI160_QMI8658C.kicad_sch (KiCad schematic)
At the start: 3 parts, among them U10 BMI160

Commit message: Changed capasitors to 0402
Parts:
- C16, C35: footprint Capacitor_SMD:C_0603_1608Metric -> Capacitor_SMD:C_0402_1005Metric
Other:
- company: (none) -> chipiki.ru
- title: (none) -> RasPi Zero NAV Hat
Changed lines of the file:
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@@
 (kicad_sch (version 20230121) (generator eeschema)
   (paper "A4" portrait)
+  (title_block
+    (title "RasPi Zero NAV Hat")
+    (date "2023-05-12")
+    (rev "0.1")
+    (company "chipiki.ru")
+    (comment 1 "RasPi Zero NAV Hat")
+    (comment 2 "Denis Tsekh")
+  )
   (junction (at 110.49 161.29) (diameter 0) (color 0 0 0 0)
   )
@@
       (effects (font (size 1.27 1.27)))
     )
-    (property "Footprint" "Capacitor_SMD:C_0603_1608Metric" (at 121.92 123.4948 0)
+    (property "Footprint" "Capacitor_SMD:C_0402_1005Metric" (at 121.92 123.4948 0)
       (effects (font (size 1.27 1.27)) hide)
     )
@@
       (effects (font (size 1.27 1.27)))
     )
-    (property "Footprint" "Capacitor_SMD:C_0603_1608Metric" (at 121.92 113.3348 0)
-      (effects (font (size 1.27 1.27)) hide)
-    )
+    (property "Footprint" "Capacitor_SMD:C_0402_1005Metric" (at 121.92 113.3348 0)
+      (effects (font (size 1.27 1.27)) hide)
+    )
