File: HW/rbpi-z-hat/QMC5883L.kicad_sch (KiCad schematic)
At the start: 6 parts, among them U6 MMC5883MA

Commit message: Apdated Sch and PCB
Parts:
- removed R13, R14: 4K7, Resistor_SMD:R_0402_1005Metric, symbol Device:R
Connections:
- net QMC_GND: now reaches C14.2, U6.11 (GND), U6.9 (GND)
- net QMC_SDA: now reaches U6.16 (SDA)
- net QMC_SCL: now reaches U6.1 (SCL)
- net QMC_INT: now reaches U6.15 (INT)
Changed lines of the file:
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@@
 (kicad_sch (version 20230121) (generator eeschema)
   (paper "A4" portrait)
-  (junction (at 97.79 151.13) (diameter 0) (color 0 0 0 0)
-  )
-  (junction (at 90.17 148.59) (diameter 0) (color 0 0 0 0)
-  )
   (junction (at 116.84 139.7) (diameter 0) (color 0 0 0 0)
-  )
-  (junction (at 90.17 130.81) (diameter 0) (color 0 0 0 0)
-  )
-  (junction (at 97.79 130.81) (diameter 0) (color 0 0 0 0)
   )
   (junction (at 114.3 162.56) (diameter 0) (color 0 0 0 0)
@@
   (junction (at 116.84 130.81) (diameter 0) (color 0 0 0 0)
   )
-  (wire (pts (xy 90.17 146.05) (xy 90.17 148.59))
-    (stroke (width 0) (type default))
-  )
-  (wire (pts (xy 90.17 148.59) (xy 104.14 148.59))
-    (stroke (width 0) (type default))
-  )
-  (wire (pts (xy 97.79 138.43) (xy 97.79 130.81))
+  (wire (pts (xy 83.82 148.59) (xy 104.14 148.59))
     (stroke (width 0) (type default))
   )
   (wire (pts (xy 114.3 139.7) (xy 116.84 139.7))
-    (stroke (width 0) (type default))
-  )
-  (wire (pts (xy 90.17 130.81) (xy 97.79 130.81))
-    (stroke (width 0) (type default))
-  )
-  (wire (pts (xy 97.79 151.13) (xy 104.14 151.13))
     (stroke (width 0) (type default))
   )
@@
     (stroke (width 0) (type default))
   )
-  (wire (pts (xy 83.82 148.59) (xy 90.17 148.59))
-    (stroke (width 0) (type default))
-  )
   (wire (pts (xy 124.46 151.13) (xy 129.54 151.13))
     (stroke (width 0) (type default))
@@
     (stroke (width 0) (type default))
   )
-  (wire (pts (xy 83.82 130.81) (xy 90.17 130.81))
-    (stroke (width 0) (type default))
-  )
-  (wire (pts (xy 90.17 138.43) (xy 90.17 130.81))
+  (wire (pts (xy 83.82 130.81) (xy 116.84 130.81))
     (stroke (width 0) (type default))
   )
@@
     (stroke (width 0) (type default))
   )
-  (wire (pts (xy 83.82 151.13) (xy 97.79 151.13))
+  (wire (pts (xy 83.82 151.13) (xy 104.14 151.13))
     (stroke (width 0) (type default))
   )
@@
     (stroke (width 0) (type default))
   )
-  (wire (pts (xy 97.79 130.81) (xy 116.84 130.81))
-    (stroke (width 0) (type default))
-  )
-  (wire (pts (xy 97.79 146.05) (xy 97.79 151.13))
-    (stroke (width 0) (type default))
-  )
   (wire (pts (xy 116.84 130.81) (xy 121.92 130.81))
     (stroke (width 0) (type default))
@@
   (text "QMC5883L" (at 116.84 146.05 0)
     (effects (font (size 1.27 1.27) (thickness 0.254) bold) (justify left bottom))
+  )
+  (hierarchical_label "QMC_SDA" (shape bidirectional) (at 83.82 151.13 180) (fields_autoplaced)
+    (effects (font (size 1.27 1.27)) (justify right))
+  )
+  (hierarchical_label "QMC_GND" (shape input) (at 83.82 162.56 180) (fields_autoplaced)
+    (effects (font (size 1.27 1.27) bold) (justify right))
+  )
+  (hierarchical_label "QMC_INT" (shape output) (at 83.82 153.67 180) (fields_autoplaced)
+    (effects (font (size 1.27 1.27)) (justify right))
+  )
+  (hierarchical_label "QMC_SCL" (shape input) (at 83.82 148.59 180) (fields_autoplaced)
+    (effects (font (size 1.27 1.27)) (justify right))
   )
   (hierarchical_label "QMC_VDD" (shape input) (at 83.82 130.81 180) (fields_autoplaced)
@@
     )
   )
-  (symbol (lib_id "Device:R") (at 97.79 142.24 0) (unit 1)
-    (in_bom yes) (on_board yes) (dnp no)
-    (property "Reference" "R14" (at 99.06 140.97 0)
-      (effects (font (size 1.27 1.27)) (justify left))
-    )
-    (property "Value" "4K7" (at 99.06 143.51 0)
-      (effects (font (size 1.27 1.27)) (justify left))
-    )
-    (property "Footprint" "Resistor_SMD:R_0402_1005Metric" (at 96.012 142.24 90)
-      (effects (font (size 1.27 1.27)) hide)
-    )
-    (property "Datasheet" "~" (at 97.79 142.24 0)
-      (effects (font (size 1.27 1.27)) hide)
-    )
-    (pin "1")
-    (pin "2")
-    (instances
-      (project "rbpi-z-hat"
-        (path "/d99b0340-d795-4b40-9cde-9851c6cee99d/740a9ed9-3c23-4e4f-8dd1-04f07ce4215e/42557423-f939-4503-bf60-cce5255c597a"
-          (reference "R14") (unit 1)
-        )
-      )
-    )
-  )
   (symbol (lib_id "Sensor_Magnetic:MMC5883MA") (at 114.3 151.13 0) (unit 1)
     (in_bom yes) (on_board yes) (dnp no)
@@
         )
       )
-    )
-  )
-  (symbol (lib_id "Device:R") (at 90.17 142.24 0) (unit 1)
-    (in_bom yes) (on_board yes) (dnp no)
-    (property "Reference" "R13" (at 91.44 140.97 0)
-      (effects (font (size 1.27 1.27)) (justify left))
-    )
-    (property "Value" "4K7" (at 91.44 143.51 0)
-      (effects (font (size 1.27 1.27)) (justify left))
-    )
-    (property "Footprint" "Resistor_SMD:R_0402_1005Metric" (at 88.392 142.24 90)
-      (effects (font (size 1.27 1.27)) hide)
-    )
-    (property "Datasheet" "~" (at 90.17 142.24 0)
-      (effects (font (size 1.27 1.27)) hide)
-    )
-    (pin "1")
-    (pin "2")
-    (instances
-      (project "rbpi-z-hat"
-        (path "/d99b0340-d795-4b40-9cde-9851c6cee99d/740a9ed9-3c23-4e4f-8dd1-04f07ce4215e/42557423-f939-4503-bf60-cce5255c597a"
-          (reference "R13") (unit 1)
-        )
-      )

Commit message: Changed capasitors to 0402
Other:
- company: (none) -> chipiki.ru
- title: (none) -> RasPi Zero NAV Hat
Changed lines of the file:
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@@
 (kicad_sch (version 20230121) (generator eeschema)
   (paper "A4" portrait)
+  (title_block
+    (title "RasPi Zero NAV Hat")
+    (date "2023-05-12")
+    (rev "0.1")
+    (company "chipiki.ru")
+    (comment 1 "RasPi Zero NAV Hat")
+    (comment 2 "Denis Tsekh")
+  )
   (junction (at 116.84 139.7) (diameter 0) (color 0 0 0 0)
   )
