File: HW/rbpi-z-hat/FerriteBeads.kicad_sch (KiCad schematic)
At the start: 4 parts

Commit message: Changes in Sch & PCB
Parts:
- L5, L6, L7, L8: footprint Inductor_SMD:L_0603_1608Metric -> Inductor_SMD:L_0402_1005Metric
Changed lines of the file:
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@@
       (effects (font (size 1.27 1.27)))
     )
-    (property "Footprint" "Inductor_SMD:L_0603_1608Metric" (at 107.95 132.588 90)
+    (property "Footprint" "Inductor_SMD:L_0402_1005Metric" (at 107.95 132.588 90)
       (effects (font (size 1.27 1.27)) hide)
     )
@@
       (effects (font (size 1.27 1.27)))
     )
-    (property "Footprint" "Inductor_SMD:L_0603_1608Metric" (at 107.95 140.208 90)
+    (property "Footprint" "Inductor_SMD:L_0402_1005Metric" (at 107.95 140.208 90)
       (effects (font (size 1.27 1.27)) hide)
     )
@@
       (effects (font (size 1.27 1.27)))
     )
-    (property "Footprint" "Inductor_SMD:L_0603_1608Metric" (at 107.95 147.828 90)
+    (property "Footprint" "Inductor_SMD:L_0402_1005Metric" (at 107.95 147.828 90)
       (effects (font (size 1.27 1.27)) hide)
     )
@@
       (effects (font (size 1.27 1.27)))
     )
-    (property "Footprint" "Inductor_SMD:L_0603_1608Metric" (at 107.95 155.448 90)
+    (property "Footprint" "Inductor_SMD:L_0402_1005Metric" (at 107.95 155.448 90)
       (effects (font (size 1.27 1.27)) hide)
     )
