File: HW/rbpi-z-hat/ICM-42688-P.kicad_sch (KiCad schematic)
At the start: 4 parts, among them U9 ICM-42688-P

Commit message: Changes in Sch & PCB
Parts:
- C28: footprint Capacitor_SMD:C_0805_2012Metric -> Capacitor_SMD:C_0603_1608Metric
- C29, C30: footprint Capacitor_SMD:C_0603_1608Metric -> Capacitor_SMD:C_0402_1005Metric
Changed lines of the file:
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@@
       (effects (font (size 1.27 1.27)))
     )
-    (property "Footprint" "Capacitor_SMD:C_0603_1608Metric" (at 101.6 116.5352 0)
+    (property "Footprint" "Capacitor_SMD:C_0402_1005Metric" (at 101.6 116.5352 0)
       (effects (font (size 1.27 1.27)) hide)
     )
@@
       (effects (font (size 1.27 1.27)))
     )
-    (property "Footprint" "Capacitor_SMD:C_0603_1608Metric" (at 125.73 114.6048 0)
+    (property "Footprint" "Capacitor_SMD:C_0402_1005Metric" (at 125.73 114.6048 0)
       (effects (font (size 1.27 1.27)) hide)
     )
@@
       (effects (font (size 1.27 1.27)))
     )
-    (property "Footprint" "Capacitor_SMD:C_0805_2012Metric" (at 125.73 104.4448 0)
+    (property "Footprint" "Capacitor_SMD:C_0603_1608Metric" (at 125.73 104.4448 0)
       (effects (font (size 1.27 1.27)) hide)
     )
