File: HW/rbpi-z-hat/I2C_CONN.kicad_sch (KiCad schematic)
At the start: 9 parts, among them J9 JST_GH, U4 PCA9306DC

Commit message: Changes in Sch & PCB
Parts:
- removed RN9: 1K5, Resistor_SMD:R_Array_Concave_4x0402, symbol Device:R_Pack04
- added R13, R14, R15, R16: 1K5, Resistor_SMD:R_0402_1005Metric, symbol Device:R
- R1: footprint Resistor_SMD:R_0603_1608Metric -> Resistor_SMD:R_0402_1005Metric
Connections:
- net +3V3: now also R13.1, R14.1, R15.1, R16.1
- net SCL: now also R13.2
- net SDA: now also R14.2
- net at D4.2 (K), J9.2 (Pin_2), U4.6 (SCL2): now also R16.2
- net at D4.1 (K), J9.3 (Pin_3), U4.5 (SDA2): now also R15.2
Changed lines of the file:
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@@
     (stroke (width 0) (type default))
   )
-  (wire (pts (xy 99.06 187.96) (xy 99.06 185.42))
+  (wire (pts (xy 99.06 182.88) (xy 99.06 187.96))
     (stroke (width 0) (type default))
   )
@@
     (stroke (width 0) (type default))
   )
-  (wire (pts (xy 96.52 185.42) (xy 96.52 187.96))
+  (wire (pts (xy 96.52 182.88) (xy 96.52 187.96))
     (stroke (width 0) (type default))
   )
@@
     (stroke (width 0) (type default))
   )
-  (wire (pts (xy 91.44 185.42) (xy 91.44 187.96))
+  (wire (pts (xy 91.44 182.88) (xy 91.44 187.96))
     (stroke (width 0) (type default))
   )
@@
     (stroke (width 0) (type default))
   )
-  (wire (pts (xy 93.98 185.42) (xy 93.98 187.96))
+  (wire (pts (xy 93.98 182.88) (xy 93.98 187.96))
     (stroke (width 0) (type default))
   )
@@
     )
   )
-  (symbol (lib_id "Device:R_Pack04") (at 93.98 180.34 180) (unit 1)
-    (in_bom yes) (on_board yes) (dnp no)
-    (property "Reference" "RN9" (at 101.6 180.34 90)
-      (effects (font (size 1.27 1.27)))
-    )
-    (property "Value" "1K5" (at 88.9 180.34 90)
-      (effects (font (size 1.27 1.27)))
-    )
-    (property "Footprint" "Resistor_SMD:R_Array_Concave_4x0402" (at 86.995 180.34 90)
-      (effects (font (size 1.27 1.27)) hide)
-    )
-    (property "Datasheet" "~" (at 93.98 180.34 0)
-      (effects (font (size 1.27 1.27)) hide)
-    )
-    (pin "1")
-    (pin "2")
-    (pin "3")
-    (pin "4")
-    (pin "5")
-    (pin "6")
-    (pin "7")
-    (pin "8")
-    (instances
-      (project "rbpi-z-hat"
-        (path "/d99b0340-d795-4b40-9cde-9851c6cee99d/00000000-0000-0000-0000-00005edd13ae"
-          (reference "RN9") (unit 1)
-        )
-      )
-    )
-  )
   (symbol (lib_id "rbpi-z-hat-rescue:+3.3V-power") (at 92.71 119.38 0) (unit 1)
     (in_bom yes) (on_board yes) (dnp no)
@@
       (effects (font (size 1.27 1.27)))
     )
-    (property "Footprint" "Resistor_SMD:R_0603_1608Metric" (at 105.918 125.73 90)
+    (property "Footprint" "Resistor_SMD:R_0402_1005Metric" (at 105.918 125.73 90)
       (effects (font (size 1.27 1.27)) hide)
     )
@@
         )
       )
+    )
+  )
+  (symbol (lib_id "Device:R") (at 91.44 179.07 180) (unit 1)
+    (in_bom yes) (on_board yes) (dnp no)
+    (property "Reference" "R13" (at 90.17 184.15 90)
+      (effects (font (size 1.27 1.27)))
+    )
+    (property "Value" "1K5" (at 91.44 179.07 90)
+      (effects (font (size 1.27 1.27)))
+    )
+    (property "Footprint" "Resistor_SMD:R_0402_1005Metric" (at 93.218 179.07 90)
+      (effects (font (size 1.27 1.27)) hide)
+    )
+    (property "Datasheet" "~" (at 91.44 179.07 0)
+      (effects (font (size 1.27 1.27)) hide)
+    )
+    (pin "1")
+    (pin "2")
+    (instances
+      (project "rbpi-z-hat"
+        (path "/d99b0340-d795-4b40-9cde-9851c6cee99d/00000000-0000-0000-0000-00005edd13ae"
+          (reference "R13") (unit 1)
+        )
+      )
+    )
+  )
+  (symbol (lib_id "Device:R") (at 96.52 179.07 180) (unit 1)
+    (in_bom yes) (on_board yes) (dnp no)
+    (property "Reference" "R15" (at 95.25 184.15 90)
+      (effects (font (size 1.27 1.27)))
+    )
+    (property "Value" "1K5" (at 96.52 179.07 90)
+      (effects (font (size 1.27 1.27)))
+    )
+    (property "Footprint" "Resistor_SMD:R_0402_1005Metric" (at 98.298 179.07 90)
+      (effects (font (size 1.27 1.27)) hide)
+    )
+    (property "Datasheet" "~" (at 96.52 179.07 0)
+      (effects (font (size 1.27 1.27)) hide)
+    )
+    (pin "1")
+    (pin "2")
+    (instances
+      (project "rbpi-z-hat"
+        (path "/d99b0340-d795-4b40-9cde-9851c6cee99d/00000000-0000-0000-0000-00005edd13ae"
+          (reference "R15") (unit 1)
+        )
+      )
+    )
+  )
+  (symbol (lib_id "Device:R") (at 93.98 179.07 180) (unit 1)
+    (in_bom yes) (on_board yes) (dnp no)
+    (property "Reference" "R14" (at 92.71 184.15 90)
+      (effects (font (size 1.27 1.27)))
+    )
+    (property "Value" "1K5" (at 93.98 179.07 90)
+      (effects (font (size 1.27 1.27)))
+    )
+    (property "Footprint" "Resistor_SMD:R_0402_1005Metric" (at 95.758 179.07 90)
+      (effects (font (size 1.27 1.27)) hide)
+    )
+    (property "Datasheet" "~" (at 93.98 179.07 0)
+      (effects (font (size 1.27 1.27)) hide)
+    )
+    (pin "1")
+    (pin "2")
+    (instances
+      (project "rbpi-z-hat"
+        (path "/d99b0340-d795-4b40-9cde-9851c6cee99d/00000000-0000-0000-0000-00005edd13ae"
+          (reference "R14") (unit 1)
+        )
+      )
+    )
+  )
+  (symbol (lib_id "Device:R") (at 99.06 179.07 180) (unit 1)
+    (in_bom yes) (on_board yes) (dnp no)
+    (property "Reference" "R16" (at 97.79 184.15 90)
+      (effects (font (size 1.27 1.27)))
+    )
+    (property "Value" "1K5" (at 99.06 179.07 90)
+      (effects (font (size 1.27 1.27)))
+    )
+    (property "Footprint" "Resistor_SMD:R_0402_1005Metric" (at 100.838 179.07 90)
+      (effects (font (size 1.27 1.27)) hide)
+    )
+    (property "Datasheet" "~" (at 99.06 179.07 0)
+      (effects (font (size 1.27 1.27)) hide)
+    )
+    (pin "1")
+    (pin "2")
+    (instances
+      (project "rbpi-z-hat"
+        (path "/d99b0340-d795-4b40-9cde-9851c6cee99d/00000000-0000-0000-0000-00005edd13ae"
+          (reference "R16") (unit 1)
+        )
+      )
