File: HW/rbpi-z-hat/BMP280.kicad_sch (KiCad schematic)
At the start: 3 parts, among them U5 BMP280

Commit message: Changed some footprints
Parts:
- C2, C4: footprint Capacitor_SMD:C_0603_1608Metric -> Capacitor_SMD:C_0402_1005Metric
Changed lines of the file:
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@@
       (effects (font (size 1.27 1.27)) (justify left))
     )
-    (property "Footprint" "Capacitor_SMD:C_0603_1608Metric" (at 141.9352 139.7 0)
+    (property "Footprint" "Capacitor_SMD:C_0402_1005Metric" (at 141.9352 139.7 0)
       (effects (font (size 1.27 1.27)) hide)
     )
@@
       (effects (font (size 1.27 1.27)) (justify left))
     )
-    (property "Footprint" "Capacitor_SMD:C_0603_1608Metric" (at 133.0452 139.7 0)
+    (property "Footprint" "Capacitor_SMD:C_0402_1005Metric" (at 133.0452 139.7 0)
       (effects (font (size 1.27 1.27)) hide)
     )
