File: HW/rbpi-z-hat/MS5611.kicad_sch (KiCad schematic)
At the start: 2 parts, among them U2 MS5611

Commit message: Changed some footprints
Parts:
- C9: footprint Capacitor_SMD:C_0603_1608Metric -> Capacitor_SMD:C_0402_1005Metric
Changed lines of the file:
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@@
       (effects (font (size 1.27 1.27)) (justify left))
     )
-    (property "Footprint" "Capacitor_SMD:C_0603_1608Metric" (at 119.0752 138.43 0)
+    (property "Footprint" "Capacitor_SMD:C_0402_1005Metric" (at 119.0752 138.43 0)
       (effects (font (size 1.27 1.27)) hide)
     )
