File: HW/rbpi-z-hat/rbpi-conn.kicad_sch (KiCad schematic)
At the start: 10 parts, among them J1 RBPI_CONN

Commit message: Changed some footprints
Parts:
- removed RN6: 10K/4x0402, Resistor_SMD:R_Array_Convex_4x0402, symbol Device:R_Pack04
- added R17, R18, R19, R20: 10K, Resistor_SMD:R_0402_1005Metric, symbol Device:R
- R11, R6: footprint Resistor_SMD:R_0603_1608Metric -> Resistor_SMD:R_0402_1005Metric
Connections:
- net +3V3: now also R17.1, R18.1, R20.1
- net GPIO_4: now also R19.2
- net SBUS_INPUT_RAW: now also R19.1
- net SCL1: now also R17.2
- net SDA1: now also R18.2

Commit message: Changed some footprints
Parts:
- removed RN5: 10K/4x0402, Resistor_SMD:R_Array_Convex_4x0402, symbol Device:R_Pack04
- added R33, R34, R35, R36: 10K, Resistor_SMD:R_0402_1005Metric, symbol Device:R
Connections:
- net Pin_11_UART_RTS is gone; now on net UART_RTS: J1.11 (Pin_11)
- net Pin_12_UART_CTS is gone; now on net UART_CTS: J1.12 (Pin_12)
- net +3V3: now also R33.1, R34.1, R35.1, R36.1
- net UART_CTS: now also R35.2
- net UART_RTS: now also R36.2
- net UART_RX: now also R33.2
- net UART_TX: now also R34.2
